Commit message: fix urdf formate

File: urdf/jetracer.urdf (robot description, URDF)
Before this commit: robot onshape, 7 links, 6 joints
Links:
- removed link body
- added link base_link, mass 1.8406011312543528735; collision mesh filename=package://jetracer_description/meshes/base_link.stl; visual mesh filename=package://jetracer_description/meshes/base_link.stl
- link wheel: mass 0.056575521129803865716 -> 0.05657552112980390735
- link wheel_2: mass 0.056575521129803865716 -> 0.05657552112980390735
- link wheel_3: mass 0.056575521129803865716 -> 0.05657552112980390735
- link wheel_4: mass 0.056575521129803865716 -> 0.05657552112980390735
Joints:
- removed joint wheel1_speed
- removed joint wheel2_speed
- removed joint wheel3_speed
- removed joint wheel4_speed
- added joint w1: type revolute, parent base_link, child wheel, origin xyz=-0.069591947474377163774 0.086073064266820473178 -4.2783187382156029344e-05 rpy=1.570796326794896558 -0 1.570796326794896336, axis 0 0 1, limit lower=0 upper=6.283185307179586232 effort=1 velocity=20
- added joint w2: type revolute, parent base_link, child wheel_2, origin xyz=0.087008052525622714413 0.086073064266820473178 -4.2783187382156029344e-05 rpy=1.570796326794896558 -0 1.57079632679489678, axis 0 0 1, limit lower=-6.283185307179586232 upper=-0 effort=1 velocity=20
- added joint w3: type revolute, parent control_arm, child wheel_3, origin xyz=-0.018299999999999996825 -2.7755575615628913511e-17 -0.01199999999999999678 rpy=-1.570796326794896336 -0 -1.570796326794896558, axis 0 0 1, limit lower=0 upper=6.283185307179586232 effort=1 velocity=20
- added joint w4: type revolute, parent control_arm_2, child wheel_4, origin xyz=-0.018300000000000010703 0 -0.012000000000000005454 rpy=1.570796326794896336 -0 1.570796326794896558, axis 0 0 1, limit lower=0 upper=6.283185307179586232 effort=1 velocity=20
- joint control_arm1: parent body -> base_link
- joint control_arm2: parent body -> base_link
