Commit message: update fix model base origin

File: urdf/original.xacro (robot description, xacro)
@@ -3,7 +3,7 @@
     <link name="Base_link">
         <inertial>
-            <origin xyz="-0.2188431446735764 0.21801110433804433 0.042341304497060785" rpy="0.0 0.0 0.0" />
-            <mass value="1.176913520449639" />
-            <inertia ixx="0.00471474301552666" iyy="0.001726030052517934" izz="0.004958600022427171" ixy="2.26448138782902e-05" iyz="0.00034033398720116436" ixz="-6.326755186562055e-05" />
+            <origin xyz="0.0016533027608847484 0.0033918428429015692 0.03234130593918531" rpy="0.0 0.0 0.0" />
+            <mass value="1.1769135204496393" />
+            <inertia ixx="0.004714734823864771" iyy="0.0017260217976734955" izz="0.004958583829422461" ixy="2.263671527874395e-05" iyz="0.0003403355352982235" ixz="-6.326913363583603e-05" />
         </inertial>
         <visual name="Base_link_visual">
@@ -22,10 +22,10 @@
     <link name="Back_left_wheel_link">
         <inertial>
-            <origin xyz="2.927331706214842e-05 0.0004286765389286629 -0.0022227221997959657" rpy="-3.944304526105059e-31 -0.0 0.0" />
-            <mass value="0.05430175599038289" />
-            <inertia ixx="1.8751279746962253e-05" iyy="1.877718038660288e-05" izz="3.0157649089595064e-05" ixy="2.1102116786955547e-09" iyz="2.4884449100952044e-08" ixz="1.7807953031446138e-09" />
+            <origin xyz="2.9305549778111394e-05 0.0004285825661594167 -0.002222785078411276" rpy="0.0 -0.0 0.0" />
+            <mass value="0.054301755990382804" />
+            <inertia ixx="1.8750879631247936e-05" iyy="1.8777013070598843e-05" izz="3.0157352809619088e-05" ixy="2.0185746688663154e-09" iyz="2.507426271228687e-08" ixz="1.7150871602248522e-09" />
         </inertial>
         <visual name="Back_left_wheel_link_visual">
-            <origin xyz="-0.018075608707960746 0.05269847562646184 0.03526135333220688" rpy="-3.141592653589791 -5.80933483705982e-14 6.103732271394052e-15" />
+            <origin xyz="-8.368700843419675e-11 -3.694822225952521e-15 4.0323300254385686e-15" rpy="-3.1415926535897913 -5.860218245151712e-14 6.1428794553838615e-15" />
             <geometry>
                 <mesh filename="meshes/Back_left_wheel_link.stl" scale="0.001 0.001 0.001" />
@@ -33,5 +33,5 @@
         </visual>
         <collision name="Back_left_wheel_link_collision">
-            <origin xyz="-0.018075608707960746 0.05269847562646184 0.03526135333220688" rpy="-3.141592653589791 -5.80933483705982e-14 6.103732271394052e-15" />
+            <origin xyz="-8.368700843419675e-11 -3.694822225952521e-15 4.0323300254385686e-15" rpy="-3.1415926535897913 -5.860218245151712e-14 6.1428794553838615e-15" />
             <geometry>
                 <mesh filename="meshes/Back_left_wheel_link.stl" scale="0.001 0.001 0.001" />
@@ -41,10 +41,10 @@
     <link name="Control_left_wheel_link">
         <inertial>
-            <origin xyz="-0.0033095632503630946 -0.0053147845774640335 0.012000000272433092" rpy="0.0 -0.0 5.4738221262687997e-48" />
-            <mass value="0.0022633439186205465" />
-            <inertia ixx="2.3321617796315383e-07" iyy="1.198225214393559e-07" izz="2.609982653238965e-07" ixy="7.588558546818485e-08" iyz="-5.316368380513131e-15" ixz="-6.531687210087995e-16" />
+            <origin xyz="-0.003309563250362881 -0.0053147845774694155 0.01200000027243138" rpy="0.0 -0.0 2.7369110631344096e-48" />
+            <mass value="0.0022633439186205456" />
+            <inertia ixx="2.3321617796315722e-07" iyy="1.1982252143935933e-07" izz="2.609982653239237e-07" ixy="7.588558546818317e-08" iyz="-5.316368380513132e-15" ixz="-6.531687210087996e-16" />
         </inertial>
         <visual name="Control_left_wheel_link_visual">
-            <origin xyz="-0.010192779328301808 -0.007691863571393674 0.012000000000000552" rpy="-3.1415926535897927 1.5707963267948903 0" />
+            <origin xyz="-0.013692779328301229 8.136428600229451e-06 0.011999999999998909" rpy="-3.1415926535897927 1.5707963267948903 0" />
             <geometry>
                 <mesh filename="meshes/Control_left_wheel_link.stl" scale="0.001 0.001 0.001" />
@@ -52,5 +52,5 @@
         </visual>
         <collision name="Control_left_wheel_link_collision">
-            <origin xyz="-0.010192779328301808 -0.007691863571393674 0.012000000000000552" rpy="-3.1415926535897927 1.5707963267948903 0" />
+            <origin xyz="-0.013692779328301229 8.136428600229451e-06 0.011999999999998909" rpy="-3.1415926535897927 1.5707963267948903 0" />
             <geometry>
                 <mesh filename="meshes/Control_left_wheel_link.stl" scale="0.001 0.001 0.001" />
@@ -60,10 +60,10 @@
     <link name="Lidar_link">
         <inertial>
-            <origin xyz="-0.028239426420145416 0.05091848444255814 6.461931578151336e-05" rpy="0.0 -0.0 5.4738221262687997e-48" />
+            <origin xyz="-0.028239426420146697 0.050918484442553716 6.461931578050084e-05" rpy="0.0 -0.0 2.7369110631344096e-48" />
             <mass value="0.08486622487588467" />
-            <inertia ixx="7.212810687965451e-05" iyy="2.7441257171711007e-05" izz="8.077472261566903e-05" ixy="-7.125364902930981e-07" iyz="-1.283711324487551e-05" ixz="-3.680051842548928e-07" />
+            <inertia ixx="7.212810687965462e-05" iyy="2.7441257171710797e-05" izz="8.077472261566897e-05" ixy="-7.125364902931029e-07" iyz="-1.2837113244875541e-05" ixz="-3.6800518425488944e-07" />
         </inertial>
         <visual name="Lidar_link_visual">
-            <origin xyz="-0.02800000439999895 0.07349999800000169 -0.009199999999996109" rpy="-3.141592653589793 -7.909058347620162e-15 1.5707963267948941" />
+            <origin xyz="-0.02800000440000023 0.07349999799999726 -0.009199999999997122" rpy="-3.141592653589793 -7.857016643340856e-15 1.5707963267948941" />
             <geometry>
                 <mesh filename="meshes/Lidar_link.stl" scale="0.001 0.001 0.001" />
@@ -71,5 +71,5 @@
         </visual>
         <collision name="Lidar_link_collision">
-            <origin xyz="-0.02800000439999895 0.07349999800000169 -0.009199999999996109" rpy="-3.141592653589793 -7.909058347620162e-15 1.5707963267948941" />
+            <origin xyz="-0.02800000440000023 0.07349999799999726 -0.009199999999997122" rpy="-3.141592653589793 -7.857016643340856e-15 1.5707963267948941" />
             <geometry>
                 <mesh filename="meshes/Lidar_link.stl" scale="0.001 0.001 0.001" />
@@ -79,10 +79,10 @@
     <link name="Front_left_wheel_link">
         <inertial>
-            <origin xyz="-0.01532972152810328 0.00042867296753681396 -2.9273400749354473e-05" rpy="1.7105694144590052e-49 -2.189528850507527e-47 0.0" />
-            <mass value="0.05430175599038289" />
-            <inertia ixx="3.0157649089595247e-05" iyy="1.8777180386603312e-05" izz="1.875127974696161e-05" ixy="2.4884449094961056e-08" iyz="-2.110211678844637e-09" ixz="-1.7807953411175636e-09" />
+            <origin xyz="-0.015329784406716503 0.00042857899476373085 -2.930563346617232e-05" rpy="0.0 -0.0 0.0" />
+            <mass value="0.05430175599038286" />
+            <inertia ixx="3.0157352809619223e-05" iyy="1.8777013070599223e-05" izz="1.8750879631248044e-05" ixy="2.5074262712313205e-08" iyz="-2.0185746688459907e-09" ixz="-1.7150871619786502e-09" />
         </inertial>
         <visual name="Front_left_wheel_link_visual">
-            <origin xyz="0.022154354003900503 0.05269847205506998 0.018075608624273445" rpy="-3.1415926535897922 1.57079632679489 0" />
+            <origin xyz="-0.013106999328301158 -3.5713994162023255e-09 -1.0902390101819038e-15" rpy="-3.1415926535897922 1.57079632679489 0" />
             <geometry>
                 <mesh filename="meshes/Front_left_wheel_link.stl" scale="0.001 0.001 0.001" />
@@ -90,5 +90,5 @@
         </visual>
         <collision name="Front_left_wheel_link_collision">
-            <origin xyz="0.022154354003900503 0.05269847205506998 0.018075608624273445" rpy="-3.1415926535897922 1.57079632679489 0" />
+            <origin xyz="-0.013106999328301158 -3.5713994162023255e-09 -1.0902390101819038e-15" rpy="-3.1415926535897922 1.57079632679489 0" />
             <geometry>
                 <mesh filename="meshes/Front_left_wheel_link.stl" scale="0.001 0.001 0.001" />
@@ -98,10 +98,10 @@
     <link name="Front_right_wheel_link">
         <inertial>
-            <origin xyz="0.015329721528106495 -0.0004286801103229632 -2.9273400749625368e-05" rpy="0.0 -0.0 0.0" />
-            <mass value="0.05430175599038288" />
-            <inertia ixx="3.0157649089595003e-05" iyy="1.8777180386602716e-05" izz="1.875127974696226e-05" ixy="2.4884449095394737e-08" iyz="2.110211678790427e-09" ixz="1.7807953408871707e-09" />
+            <origin xyz="0.01532978440671709 -0.00042858613756155964 -2.9305633465739334e-05" rpy="0.0 -0.0 0.0" />
+            <mass value="0.05430175599038282" />
+            <inertia ixx="3.0157352809619088e-05" iyy="1.8777013070598897e-05" izz="1.8750879631247827e-05" ixy="2.5074262712421625e-08" iyz="2.0185746688392145e-09" ixz="1.715087161843125e-09" />
         </inertial>
         <visual name="Front_right_wheel_link_visual">
-            <origin xyz="-0.022154354003896773 -0.05269847919785653 0.01807560862427293" rpy="-5.855923348111018e-15 1.570796326794886 0" />
+            <origin xyz="0.013106999328301764 -3.5713984747332006e-09 -5.795364188543317e-16" rpy="-5.855923348111018e-15 1.570796326794886 0" />
             <geometry>
                 <mesh filename="meshes/Front_right_wheel_link.stl" scale="0.001 0.001 0.001" />
@@ -109,5 +109,5 @@
         </visual>
         <collision name="Front_right_wheel_link_collision">
-            <origin xyz="-0.022154354003896773 -0.05269847919785653 0.01807560862427293" rpy="-5.855923348111018e-15 1.570796326794886 0" />
+            <origin xyz="0.013106999328301764 -3.5713984747332006e-09 -5.795364188543317e-16" rpy="-5.855923348111018e-15 1.570796326794886 0" />
             <geometry>
                 <mesh filename="meshes/Front_right_wheel_link.stl" scale="0.001 0.001 0.001" />
@@ -117,10 +117,10 @@
     <link name="Back_right_wheel_link">
         <inertial>
-            <origin xyz="-2.927348443597877e-05 0.00042867653892818324 0.0022227221998004864" rpy="3.944304526105059e-31 -0.0 0.0" />
-            <mass value="0.054301755990382755" />
-            <inertia ixx="1.8751279746962144e-05" iyy="1.877718038660288e-05" izz="3.0157649089595227e-05" ixy="-2.110211679820415e-09" iyz="-2.4884449095749382e-08" ixz="1.7807953431086937e-09" />
+            <origin xyz="-2.9305717152134926e-05 0.0004285825661590259 0.002222785078411231" rpy="0.0 -0.0 0.0" />
+            <mass value="0.05430175599038278" />
+            <inertia ixx="1.8750879631247827e-05" iyy="1.877701307059868e-05" izz="3.0157352809619142e-05" ixy="-2.018574668947631e-09" iyz="-2.5074262712396793e-08" ixz="1.7150871637732448e-09" />
         </inertial>
         <visual name="Back_right_wheel_link_visual">
-            <origin xyz="0.018075608540586076 0.05269847562646175 -0.035261353332204315" rpy="-1.1782268753097997e-15 -5.899896782659704e-14 -3.1415926535897873" />
+            <origin xyz="-8.368699067062835e-11 -4.0145664570445665e-15 -4.076738946423575e-15" rpy="-1.122715724078533e-15 -5.83598131927346e-14 -3.1415926535897873" />
             <geometry>
                 <mesh filename="meshes/Back_right_wheel_link.stl" scale="0.001 0.001 0.001" />
@@ -128,5 +128,5 @@
         </visual>
         <collision name="Back_right_wheel_link_collision">
-            <origin xyz="0.018075608540586076 0.05269847562646175 -0.035261353332204315" rpy="-1.1782268753097997e-15 -5.899896782659704e-14 -3.1415926535897873" />
+            <origin xyz="-8.368699067062835e-11 -4.0145664570445665e-15 -4.076738946423575e-15" rpy="-1.122715724078533e-15 -5.83598131927346e-14 -3.1415926535897873" />
             <geometry>
                 <mesh filename="meshes/Back_right_wheel_link.stl" scale="0.001 0.001 0.001" />
@@ -136,10 +136,10 @@
     <link name="Control_right_wheel_link">
         <inertial>
-            <origin xyz="0.003309563250364711 -0.005314784577464096 0.011999999727568005" rpy="0.0 -0.0 5.4738221262687997e-48" />
-            <mass value="0.0022633439186205465" />
-            <inertia ixx="2.3321617796315383e-07" iyy="1.198225214393576e-07" izz="2.6099826532390326e-07" ixy="-7.588558546818485e-08" iyz="5.316368019691282e-15" ixz="-6.531691108253035e-16" />
+            <origin xyz="0.0033095632503634675 -0.005314784577468403 0.011999999727566987" rpy="0.0 -0.0 2.7369110631344096e-48" />
+            <mass value="0.0022633439186205456" />
+            <inertia ixx="2.3321617796315722e-07" iyy="1.1982252143936103e-07" izz="2.609982653239169e-07" ixy="-7.588558546818486e-08" iyz="5.316368019691284e-15" ixz="-6.531691108253036e-16" />
         </inertial>
         <visual name="Control_right_wheel_link_visual">
-            <origin xyz="0.010192779328303425 -0.007691863571393745 0.012000000000000451" rpy="3.1415926535897927 -1.5707963267948855 0" />
+            <origin xyz="0.013692779328301815 8.1364286015706e-06 0.01199999999999946" rpy="3.1415926535897913 -1.5707963267948855 0" />
             <geometry>
                 <mesh filename="meshes/Control_right_wheel_link.stl" scale="0.001 0.001 0.001" />
@@ -147,5 +147,5 @@
         </visual>
         <collision name="Control_right_wheel_link_collision">
-            <origin xyz="0.010192779328303425 -0.007691863571393745 0.012000000000000451" rpy="3.1415926535897927 -1.5707963267948855 0" />
+            <origin xyz="0.013692779328301815 8.1364286015706e-06 0.01199999999999946" rpy="3.1415926535897913 -1.5707963267948855 0" />
             <geometry>
                 <mesh filename="meshes/Control_right_wheel_link.stl" scale="0.001 0.001 0.001" />
@@ -154,11 +154,11 @@
     </link>
     <joint name="Control_left_joint" type="continuous">
-        <origin xyz="-0.28049647923282217 0.27461929244593714 0.035799999999999846" rpy="3.141592653589785 1.0191500421363112e-16 -7.546047120498976e-16" />
+        <origin xyz="-0.06000000000000318 0.06000000000000318 0.025799999999999795" rpy="3.141592653589785 7.762887554995295e-17 -2.0933157334479724e-15" />
         <parent link="Base_link" />
         <child link="Control_left_wheel_link" />
-        <axis xyz="2.465190328815662e-32 2.2204460492503136e-16 0.9999999999999999" />
+        <axis xyz="1.232595164407831e-32 2.220446049250314e-16 1.0" />
     </joint>
     <joint name="Back_left_wheel_joint" type="continuous">
-        <origin xyz="-0.2987964792328232 0.12461929244592986 0.025298850000000938" rpy="3.14159265358979 -1.5707963267948906 0" />
+        <origin xyz="-0.07830000000000438 -0.09000000000000409 0.015298850000000884" rpy="3.1415926535897887 -1.5707963267948906 0" />
         <parent link="Base_link" />
         <child link="Back_left_wheel_link" />
@@ -166,11 +166,11 @@
     </joint>
     <joint name="Front_left_wheel_joint" type="continuous">
-        <origin xyz="-0.005192780000000008 8.140000000018687e-06 0.012000000000000002" rpy="-2.2204460492503136e-16 -1.7256332301709638e-31 -6.783780320957819e-32" />
+        <origin xyz="-0.005192779999999999 8.140000000009807e-06 0.012000000000000002" rpy="-2.220446049250314e-16 1.2325951644078504e-32 8.712952773709936e-31" />
         <parent link="Control_left_wheel_link" />
         <child link="Front_left_wheel_link" />
-        <axis xyz="0.9999999999999999 0.0 0.0" />
+        <axis xyz="1.0 0.0 0.0" />
     </joint>
     <joint name="Back_right_wheel_joint" type="continuous">
-        <origin xyz="-0.14219647923281456 0.12461929244592974 0.025298850000000928" rpy="-3.141592653589792 -1.5707963267948906 0" />
+        <origin xyz="0.07830000000000423 -0.09000000000000441 0.01529885000000087" rpy="-3.141592653589793 -1.5707963267948906 0" />
         <parent link="Base_link" />
         <child link="Back_right_wheel_link" />
@@ -178,17 +178,17 @@
     </joint>
     <joint name="Front_right_wheel_joint" type="continuous">
-        <origin xyz="0.005192780000000008 8.140000000018687e-06 0.012000000000000002" rpy="-2.2204460492503136e-16 2.4651903288156605e-32 -6.783780320957824e-32" />
+        <origin xyz="0.005192779999999999 8.140000000009807e-06 0.012000000000000002" rpy="-2.2204460492503155e-16 1.2325951644078153e-32 -7.064265330710301e-31" />
         <parent link="Control_right_wheel_link" />
         <child link="Front_right_wheel_link" />
-        <axis xyz="-0.9999999999999999 0.0 0.0" />
+        <axis xyz="-1.0 0.0 0.0" />
     </joint>
     <joint name="Control_right_joint" type="continuous">
-        <origin xyz="-0.1604964792328156 0.274619292445937 0.03579999999999983" rpy="3.141592653589785 1.0191500421363112e-16 -7.546047120498976e-16" />
+        <origin xyz="0.06000000000000339 0.06000000000000293 0.02579999999999979" rpy="3.141592653589785 7.762887554995295e-17 -2.0933157334479724e-15" />
         <parent link="Base_link" />
         <child link="Control_right_wheel_link" />
-        <axis xyz="2.465190328815662e-32 2.2204460492503136e-16 0.9999999999999999" />
+        <axis xyz="1.232595164407831e-32 2.220446049250314e-16 1.0" />
     </joint>
     <joint name="Lidar_joint" type="fixed">
-        <origin xyz="-0.19249651923281735 0.2476192424459362 0.10997548000000107" rpy="3.141592653589785 1.0191500421363112e-16 -7.546047120498976e-16" />
+        <origin xyz="0.0279999600000016 0.032999950000002144 0.09997548000000103" rpy="3.141592653589785 7.762887554995295e-17 -2.0933157334479724e-15" />
         <parent link="Base_link" />
         <child link="Lidar_link" />
