Commit message: fix urdf

File: urdf/jetracer_joints.xacro (robot description, xacro)
@@ -15,16 +15,21 @@
         </joint>
     </xacro:macro>
+    <joint name="chassis_joint" type="fixed">
+    <origin xyz="0 0 0" rpy="0 0 0" />
+    <parent link="base_link" />
+    <child link="chassis_link" />
+  </joint>
     <!-- ================ JOINTS ================ -->
-    <xacro:joint joint_name="Back_left_wheel_joint" parent_name="base_link" child_name="Back_left_wheel_link" joint_type="continuous" >
+    <xacro:joint joint_name="Back_left_wheel_joint" parent_name="chassis_link" child_name="Back_left_wheel_link" joint_type="continuous" >
         <origin xyz="-0.07830000000000438 -0.09000000000000409 0.015298850000000884" rpy="3.1415926535897887 -1.5707963267948906 0" />
         <axis xyz="0.0 -2.303712776096894e-15 1.0" />
         <limit/>
     </xacro:joint>
-    <xacro:joint joint_name="Back_right_wheel_joint" parent_name="base_link" child_name="Back_right_wheel_link" joint_type="continuous" >
+    <xacro:joint joint_name="Back_right_wheel_joint" parent_name="chassis_link" child_name="Back_right_wheel_link" joint_type="continuous" >
         <origin xyz="0.07830000000000423 -0.09000000000000441 0.01529885000000087" rpy="-3.141592653589793 -1.5707963267948906 0" />
         <axis xyz="0.0 2.1926904736343785e-15 1.0" />
         <limit/>
     </xacro:joint>
-    <xacro:joint joint_name="Control_left_joint" parent_name="base_link" child_name="Control_left_wheel_link" joint_type="revolute" >
+    <xacro:joint joint_name="Control_left_joint" parent_name="chassis_link" child_name="Control_left_wheel_link" joint_type="revolute" >
         <origin xyz="-0.06000000000000318 0.06000000000000318 0.025799999999999795" rpy="3.141592653589785 7.762887554995295e-17 -2.0933157334479724e-15" />
         <axis xyz="1.232595164407831e-32 2.220446049250314e-16 1.0" />
@@ -36,5 +41,5 @@
         <limit/>
     </xacro:joint>
-    <xacro:joint joint_name="Control_right_joint" parent_name="base_link" child_name="Control_right_wheel_link" joint_type="revolute" >
+    <xacro:joint joint_name="Control_right_joint" parent_name="chassis_link" child_name="Control_right_wheel_link" joint_type="revolute" >
         <origin xyz="0.06000000000000339 0.06000000000000293 0.02579999999999979" rpy="3.141592653589785 7.762887554995295e-17 -2.0933157334479724e-15" />
         <axis xyz="1.232595164407831e-32 2.220446049250314e-16 1.0" />
@@ -46,5 +51,5 @@
         <limit/>
     </xacro:joint>
-    <xacro:joint joint_name="Lidar_joint" parent_name="base_link" child_name="Lidar_link" joint_type="fixed" >
+    <xacro:joint joint_name="Lidar_joint" parent_name="chassis_link" child_name="Lidar_link" joint_type="fixed" >
         <origin xyz="0.0279999600000016 0.032999950000002144 0.09997548000000103" rpy="3.141592653589785 7.762887554995295e-17 -2.0933157334479724e-15" />
         <axis/>

File: urdf/jetracer_links.xacro (robot description, xacro)
@@ -21,7 +21,8 @@
         </link>
     </xacro:macro>
+    <link name="base_link" />
     <!-- ================ JOINTS ================ -->
-    <!-- base link -->
-    <xacro:links name="base_link" mesh="${base_link_mesh}" material="${base_link_material}" mass="${base_link_mass}">
+    <!-- chassis link -->
+    <xacro:links name="chassis_link" mesh="${chassis_link_mesh}" material="${chassis_link_material}" mass="${chassis_link_mass}">
         <origin xyz="0.0 0.0 0.0" rpy="0.0 0.0 0.0" />
         <inertial>

File: urdf/jetracer_main.xacro (robot description, xacro)
@@ -4,5 +4,5 @@
     <xacro:property name="scale" value="0.001 0.001 0.001" />
     <!-- ==== meshes ==== -->
-    <xacro:property name="base_link_mesh"               value="file://$(find jetracer_description)/meshes/Base_link.stl" />
+    <xacro:property name="chassis_link_mesh"               value="file://$(find jetracer_description)/meshes/Base_link.stl" />
     <!-- Rear -->
     <xacro:property name="Back_left_wheel_mesh"         value="file://$(find jetracer_description)/meshes/Back_left_wheel_link.stl" />
@@ -15,5 +15,5 @@
     <xacro:property name="Lidar_mesh"                   value="file://$(find jetracer_description)/meshes/Lidar_link.stl" />
     <!-- ==== materials ==== -->
-    <xacro:property name="base_link_material"           value="0.25 0.25 0.25 1" />
+    <xacro:property name="chassis_link_material"           value="0.25 0.25 0.25 1" />
     <!-- Rear -->
     <xacro:property name="Back_left_wheel_material"     value="0.5 0.5 0.4 1" />
@@ -26,5 +26,5 @@
     <xacro:property name="Lidar_material"               value="0.5 0.5 0.4 1" />
     <!-- ==== mass ==== -->
-    <xacro:property name="base_link_mass"               value="1.176913520449639" />
+    <xacro:property name="chassis_link_mass"               value="1.176913520449639" />
     <!-- Rear -->
     <xacro:property name="Back_left_wheel_mass"         value="0.05430175599038289" />

File: urdf/jetracer_sensors.xacro (robot description, xacro)
@@ -18,13 +18,23 @@
             <command_interface name="position" />
             <state_interface name="position" />
+            <state_interface name="velocity" />
         </joint>
         <joint name="Control_right_joint">
             <command_interface name="position" />
             <state_interface name="position" />
+            <state_interface name="velocity" />
+        </joint>
+        <joint name="Front_left_wheel_joint">
+            <state_interface name="velocity"/>
+            <state_interface name="position"/>
+        </joint>
+        <joint name="Front_right_wheel_joint">
+            <state_interface name="velocity"/>
+            <state_interface name="position"/>
         </joint>
     </ros2_control>
     <gazebo>
         <plugin filename="gz_ros2_control-system" name="gz_ros2_control::GazeboSimROS2ControlPlugin">
-        <parameters>$(find gz_ros2_control_demos)/config/ackermann_drive_controller.yaml</parameters>
+        <parameters>$(find jetracer_description)/config/jetracer_controller.yaml</parameters>
         </plugin>
   </gazebo>

Commit message: fix back joint direction

File: urdf/jetracer_joints.xacro (robot description, xacro)
@@ -23,10 +23,10 @@
     <xacro:joint joint_name="Back_left_wheel_joint" parent_name="chassis_link" child_name="Back_left_wheel_link" joint_type="continuous" >
         <origin xyz="-0.07830000000000438 -0.09000000000000409 0.015298850000000884" rpy="3.1415926535897887 -1.5707963267948906 0" />
-        <axis xyz="0.0 -2.303712776096894e-15 1.0" />
+        <axis xyz="0.0 -2.303712776096894e-15 -1.0" />
         <limit/>
     </xacro:joint>
     <xacro:joint joint_name="Back_right_wheel_joint" parent_name="chassis_link" child_name="Back_right_wheel_link" joint_type="continuous" >
         <origin xyz="0.07830000000000423 -0.09000000000000441 0.01529885000000087" rpy="-3.141592653589793 -1.5707963267948906 0" />
-        <axis xyz="0.0 2.1926904736343785e-15 1.0" />
+        <axis xyz="0.0 2.1926904736343785e-15 -1.0" />
         <limit/>
     </xacro:joint>

File: urdf/jetracer_sensors.xacro (robot description, xacro)
@@ -36,5 +36,5 @@
     <gazebo>
         <plugin filename="gz_ros2_control-system" name="gz_ros2_control::GazeboSimROS2ControlPlugin">
-        <parameters>$(find jetracer_description)/config/jetracer_controller.yaml</parameters>
+            <parameters>$(find jetracer_description)/config/jetracer_controller.yaml</parameters>
         </plugin>
   </gazebo>

Commit message: fix robot orientation

File: urdf/jetracer_joints.xacro (robot description, xacro)
@@ -22,35 +22,35 @@
     <!-- ================ JOINTS ================ -->
     <xacro:joint joint_name="Back_left_wheel_joint" parent_name="chassis_link" child_name="Back_left_wheel_link" joint_type="continuous" >
-        <origin xyz="-0.07830000000000438 -0.09000000000000409 0.015298850000000884" rpy="3.1415926535897887 -1.5707963267948906 0" />
-        <axis xyz="0.0 -2.303712776096894e-15 -1.0" />
+        <origin xyz="-0.08999999999999997 0.07830000000000013 0.015298849999999503" rpy="1.5707963267949487 -9.036958300754793e-32 -5.096753522204392e-16" />
+        <axis xyz="-2.0095106667766018e-44 5.847752837517865e-14 1.0" />
         <limit/>
     </xacro:joint>
     <xacro:joint joint_name="Back_right_wheel_joint" parent_name="chassis_link" child_name="Back_right_wheel_link" joint_type="continuous" >
-        <origin xyz="0.07830000000000423 -0.09000000000000441 0.01529885000000087" rpy="-3.141592653589793 -1.5707963267948906 0" />
-        <axis xyz="0.0 2.1926904736343785e-15 -1.0" />
+        <origin xyz="-0.09000000000000004 -0.07829999999999988 0.015298850000000502" rpy="1.5707963267948317 -9.036958300754793e-32 -5.096753522204392e-16" />
+        <axis xyz="-2.0095106667766018e-44 -5.848446726908255e-14 1.0" />
         <limit/>
     </xacro:joint>
     <xacro:joint joint_name="Control_left_joint" parent_name="chassis_link" child_name="Control_left_wheel_link" joint_type="revolute" >
-        <origin xyz="-0.06000000000000318 0.06000000000000318 0.025799999999999795" rpy="3.141592653589785 7.762887554995295e-17 -2.0933157334479724e-15" />
-        <axis xyz="1.232595164407831e-32 2.220446049250314e-16 1.0" />
+        <origin xyz="0.060000000000000026 0.060000000000000116 0.02579999999999962" rpy="3.141592653589787 -9.036958300754793e-32 -5.096753522204392e-16" />
+        <axis xyz="0.0 -3.469446951953671e-18 1.0" />
         <limit lower="-${PI/2}" upper="${PI/2}" effort="1000000" velocity="1000000" />
     </xacro:joint>
     <xacro:joint joint_name="Front_left_wheel_joint" parent_name="Control_left_wheel_link" child_name="Front_left_wheel_link" joint_type="continuous" >
-        <origin xyz="-0.005192779999999999 8.140000000009807e-06 0.012000000000000002" rpy="-2.220446049250314e-16 1.2325951644078504e-32 8.712952773709936e-31" />
-        <axis xyz="1.0 0.0 0.0" />
+        <origin xyz="-8.140000000009807e-06 0.005192779999999999 0.012000000000000002" rpy="3.469446951953529e-18 3.944304526105059e-31 2.0096475123297585e-44" />
+        <axis xyz="0.0 -1.0 -3.1672338534784104e-31" />
         <limit/>
     </xacro:joint>
     <xacro:joint joint_name="Control_right_joint" parent_name="chassis_link" child_name="Control_right_wheel_link" joint_type="revolute" >
-        <origin xyz="0.06000000000000339 0.06000000000000293 0.02579999999999979" rpy="3.141592653589785 7.762887554995295e-17 -2.0933157334479724e-15" />
-        <axis xyz="1.232595164407831e-32 2.220446049250314e-16 1.0" />
+        <origin xyz="0.05999999999999998 -0.05999999999999989 0.02580000000000038" rpy="3.141592653589787 -9.036958300754793e-32 -5.096753522204392e-16" />
+        <axis xyz="0.0 -3.469446951953671e-18 1.0" />
         <limit lower="-${PI/2}" upper="${PI/2}" effort="1000000" velocity="1000000" />
     </xacro:joint>
     <xacro:joint joint_name="Front_right_wheel_joint" parent_name="Control_right_wheel_link" child_name="Front_right_wheel_link" joint_type="continuous" >
-        <origin xyz="0.005192779999999999 8.140000000009807e-06 0.012000000000000002" rpy="-2.2204460492503155e-16 1.2325951644078153e-32 -7.064265330710301e-31" />
-        <axis xyz="-1.0 0.0 0.0" />
+        <origin xyz="-8.140000000009807e-06 0.005192779999999999 0.012000000000000002" rpy="3.469446951953529e-18 3.944304526105059e-31 2.0096475123297585e-44" />
+        <axis xyz="0.0 -1.0 -3.1672338534784104e-31" />
         <limit/>
     </xacro:joint>
     <xacro:joint joint_name="Lidar_joint" parent_name="chassis_link" child_name="Lidar_link" joint_type="fixed" >
-        <origin xyz="0.0279999600000016 0.032999950000002144 0.09997548000000103" rpy="3.141592653589785 7.762887554995295e-17 -2.0933157334479724e-15" />
+        <origin xyz="0.032999949999999986 -0.027999959999999404 0.09997548000000019" rpy="3.141592653589787 -9.036958300754793e-32 -5.096753522204392e-16" />
         <axis/>
         <limit/>

File: urdf/jetracer_links.xacro (robot description, xacro)
@@ -27,70 +27,70 @@
         <origin xyz="0.0 0.0 0.0" rpy="0.0 0.0 0.0" />
         <inertial>
-            <origin xyz="0.0016533027608847484 0.0033918428429015692 0.03234130593918531" rpy="0.0 0.0 0.0" />
+            <origin xyz="0.003391842842901498 -0.0016533027608844348 0.03234130593918586" rpy="0.0 0.0 0.0" />
             <mass value="1.1769135204496393" />
-            <inertia ixx="0.004714734823864771" iyy="0.0017260217976734955" izz="0.004958583829422461" ixy="2.263671527874395e-05" iyz="0.0003403355352982235" ixz="-6.326913363583603e-05" />
+            <inertia ixx="0.0017260217976737531" iyy="0.004714734823865151" izz="0.0049585838294225635" ixy="-2.263671527874525e-05" iyz="6.326913363584177e-05" ixz="0.0003403355352982155" />
         </inertial>
     </xacro:links>
     <!-- Rear left wheel link -->
     <xacro:links name="Back_left_wheel_link" mesh="${Back_left_wheel_mesh}" material="${Back_left_wheel_material}" mass="${Back_left_wheel_mass}">
-        <origin xyz="-8.368700843419675e-11 -3.694822225952521e-15 4.0323300254385686e-15" rpy="-3.1415926535897913 -5.860218245151712e-14 6.1428794553838615e-15" />
+        <origin xyz="-3.375077994860476e-16 -8.368559845095547e-11 -3.019806626980426e-16" rpy="-3.141592653589788 -2.2183649806874918e-15 -2.1736792697780755e-29" />
         <inertial>
-            <origin xyz="2.9305549778111394e-05 0.0004285825661594167 -0.002222785078411276" rpy="0.0 -0.0 0.0" />
+            <origin xyz="2.9305633464797864e-05 0.0004285824824775064 -0.002222785078415628" rpy="0.0 -0.0 0.0" />
             <mass value="0.054301755990382804" />
-            <inertia ixx="1.8750879631247936e-05" iyy="1.8777013070598843e-05" izz="3.0157352809619088e-05" ixy="2.0185746688663154e-09" iyz="2.507426271228687e-08" ixz="1.7150871602248522e-09" />
+            <inertia ixx="1.8750879631247773e-05" iyy="1.8777013070598843e-05" izz="3.0157352809619304e-05" ixy="2.018574668879972e-09" iyz="2.5074262712355275e-08" ixz="1.7150871619786058e-09" />
         </inertial>
     </xacro:links>
     <!-- Rear right wheel link -->
     <xacro:links name="Back_right_wheel_link" mesh="${Back_right_wheel_link}" material="${Back_right_wheel_material}" mass="${Back_right_wheel_mass}">
-        <origin xyz="-8.368699067062835e-11 -4.0145664570445665e-15 -4.076738946423575e-15" rpy="-1.122715724078533e-15 -5.83598131927346e-14 -3.1415926535897873" />
+        <origin xyz="-3.375077994860476e-16 -8.368659543123158e-11 2.1316282072803005e-16" rpy="-5.397793497891479e-15 -2.2780382690294677e-15 3.141592653589793" />
         <inertial>
-            <origin xyz="-2.9305717152134926e-05 0.0004285825661590259 0.002222785078411231" rpy="0.0 -0.0 0.0" />
+            <origin xyz="-2.930563346547288e-05 0.0004285824824764406 0.0022227850784155034" rpy="0.0 -0.0 0.0" />
             <mass value="0.05430175599038278" />
-            <inertia ixx="1.8750879631247827e-05" iyy="1.877701307059868e-05" izz="3.0157352809619142e-05" ixy="-2.018574668947631e-09" iyz="-2.5074262712396793e-08" ixz="1.7150871637732448e-09" />
+            <inertia ixx="1.8750879631247936e-05" iyy="1.877701307059906e-05" izz="3.0157352809619033e-05" ixy="-2.018574668947735e-09" iyz="-2.5074262712517995e-08" ixz="1.7150871620087073e-09" />
         </inertial>
     </xacro:links>
     <!-- Front left control link -->
     <xacro:links name="Control_left_wheel_link" mesh="${Control_left_wheel_link}" material="${Control_left_wheel_material}" mass="${Control_left_wheel_mass}">
-        <origin xyz="-0.013692779328301229 8.136428600229451e-06 0.011999999999998909" rpy="-3.1415926535897927 1.5707963267948903 0" />
+        <origin xyz="-8.136428598293222e-06 -0.013692779328306655 0.011999999999999334" rpy="1.570796326794897 1.5707963267948903 0" />
         <inertial>
-            <origin xyz="-0.003309563250362881 -0.0053147845774694155 0.01200000027243138" rpy="0.0 -0.0 2.7369110631344096e-48" />
+            <origin xyz="0.005314784577471352 -0.003309563250368317 0.012000000272431918" rpy="0.0 -0.0 0.0" />
             <mass value="0.0022633439186205456" />
-            <inertia ixx="2.3321617796315722e-07" iyy="1.1982252143935933e-07" izz="2.609982653239237e-07" ixy="7.588558546818317e-08" iyz="-5.316368380513132e-15" ixz="-6.531687210087996e-16" />
+            <inertia ixx="1.1982252143935764e-07" iyy="2.3321617796315213e-07" izz="2.609982653239135e-07" ixy="-7.588558546818486e-08" iyz="-6.531687219143192e-16" ixz="5.316366320884021e-15" />
         </inertial>
     </xacro:links>
     <!-- Front left wheel link -->
     <xacro:links name="Front_left_wheel_link" mesh="${Front_left_wheel_mesh}" material="${Front_left_wheel_material}" mass="${Front_left_wheel_mass}">
-        <origin xyz="-0.013106999328301158 -3.5713994162023255e-09 -1.0902390101819038e-15" rpy="-3.1415926535897922 1.57079632679489 0" />
+        <origin xyz="3.571401290258791e-09 -0.013106999328306461 -4.019007349143067e-16" rpy="1.570796326794896 1.5707963267948843 0" />
         <inertial>
-            <origin xyz="-0.015329784406716503 0.00042857899476373085 -2.930563346617232e-05" rpy="0.0 -0.0 0.0" />
+            <origin xyz="-0.0004285789947618479 -0.015329784406721796 -2.930563346551729e-05" rpy="0.0 -0.0 1.4597325655620378e-62" />
             <mass value="0.05430175599038286" />
-            <inertia ixx="3.0157352809619223e-05" iyy="1.8777013070599223e-05" izz="1.8750879631248044e-05" ixy="2.5074262712313205e-08" iyz="-2.0185746688459907e-09" ixz="-1.7150871619786502e-09" />
+            <inertia ixx="1.8777013070599114e-05" iyy="3.0157352809619142e-05" izz="1.8750879631248044e-05" ixy="-2.5074262712421625e-08" iyz="-1.71508716181602e-09" ixz="2.0185746688459907e-09" />
         </inertial>
     </xacro:links>
     <!-- Front right control link -->
     <xacro:links name="Control_right_wheel_link" mesh="${Control_right_wheel_link}" material="${Control_right_wheel_material}" mass="${Control_right_wheel_mass}">
-        <origin xyz="0.013692779328301815 8.1364286015706e-06 0.01199999999999946" rpy="3.1415926535897913 -1.5707963267948855 0" />
+        <origin xyz="-8.136428598666257e-06 0.013692779328305269 0.012000000000000144" rpy="-1.5707963267948972 -1.570796326794894 0" />
         <inertial>
-            <origin xyz="0.0033095632503634675 -0.005314784577468403 0.011999999727566987" rpy="0.0 -0.0 2.7369110631344096e-48" />
+            <origin xyz="0.005314784577471317 0.0033095632503669314 0.011999999727567632" rpy="0.0 -0.0 0.0" />
             <mass value="0.0022633439186205456" />
-            <inertia ixx="2.3321617796315722e-07" iyy="1.1982252143936103e-07" izz="2.609982653239169e-07" ixy="-7.588558546818486e-08" iyz="5.316368019691284e-15" ixz="-6.531691108253036e-16" />
+            <inertia ixx="1.1982252143936103e-07" iyy="2.3321617796315552e-07" izz="2.609982653239203e-07" ixy="7.588558546818486e-08" iyz="-6.531695352472969e-16" ixz="-5.3163683852545e-15" />
         </inertial>
     </xacro:links>
     <!-- Front right wheel link -->
     <xacro:links name="Front_right_wheel_link" mesh="${Front_right_wheel_link}" material="${Front_right_wheel_material}" mass="${Front_right_wheel_mass}">
-        <origin xyz="0.013106999328301764 -3.5713984747332006e-09 -5.795364188543317e-16" rpy="-5.855923348111018e-15 1.570796326794886 0" />
+        <origin xyz="3.5714013080223594e-09 0.01310699932830512 -3.3084646133829665e-16" rpy="-1.5707963267949037 1.5707963267948886 0" />
         <inertial>
-            <origin xyz="0.01532978440671709 -0.00042858613756155964 -2.9305633465739334e-05" rpy="0.0 -0.0 0.0" />
+            <origin xyz="0.00042858613756439293 0.015329784406720446 -2.9305633465488423e-05" rpy="0.0 -0.0 0.0" />
             <mass value="0.05430175599038282" />
-            <inertia ixx="3.0157352809619088e-05" iyy="1.8777013070598897e-05" izz="1.8750879631247827e-05" ixy="2.5074262712421625e-08" iyz="2.0185746688392145e-09" ixz="1.715087161843125e-09" />
+            <inertia ixx="1.877701307059895e-05" iyy="3.015735280961906e-05" izz="1.8750879631247827e-05" ixy="-2.5074262712475835e-08" iyz="1.715087161843125e-09" ixz="-2.0185746688459907e-09" />
         </inertial>
     </xacro:links>
     <!-- Lidar link -->
     <xacro:links name="Lidar_link" mesh="${Lidar_mesh}" material="${Lidar_material}" mass="${Lidar_mass}">
-        <origin xyz="-0.02800000440000023 0.07349999799999726 -0.009199999999997122" rpy="-3.141592653589793 -7.857016643340856e-15 1.5707963267948941" />
+        <origin xyz="-0.07349999799999639 -0.028000004399998054 -0.009199999999999786" rpy="3.1415926535897225 -1.936181792881828e-15 3.1415926535897927" />
         <inertial>
-            <origin xyz="-0.028239426420146697 0.050918484442553716 6.461931578050084e-05" rpy="0.0 -0.0 2.7369110631344096e-48" />
+            <origin xyz="-0.050918484442552904 -0.028239426420145132 6.461931577792513e-05" rpy="0.0 -0.0 0.0" />
             <mass value="0.08486622487588467" />
-            <inertia ixx="7.212810687965462e-05" iyy="2.7441257171710797e-05" izz="8.077472261566897e-05" ixy="-7.125364902931029e-07" iyz="-1.2837113244875541e-05" ixz="-3.6800518425488944e-07" />
+            <inertia ixx="2.7441257171710587e-05" iyy="7.212810687965462e-05" izz="8.077472261566907e-05" ixy="7.125364902921147e-07" iyz="-3.6800518425547077e-07" ixz="1.2837113244875235e-05" />
         </inertial>
     </xacro:links>
