Commit message: fix orientation

File: urdf/jetracer_joints.xacro (robot description, xacro)
@@ -22,35 +22,35 @@
     <!-- ================ JOINTS ================ -->
     <xacro:joint joint_name="Back_left_wheel_joint" parent_name="chassis_link" child_name="Back_left_wheel_link" joint_type="continuous" >
-        <origin xyz="-0.08999999999999997 0.07830000000000013 0.015298849999999503" rpy="1.5707963267949487 -9.036958300754793e-32 -5.096753522204392e-16" />
-        <axis xyz="-2.0095106667766018e-44 5.847752837517865e-14 1.0" />
+        <origin xyz="0.0899999999999996 -0.07830000000000042 0.015298849999999736" rpy="-1.5707963267949614 -4.7336595440742014e-32 -3.872106723056806e-16" />
+        <axis xyz="1.5368552462246833e-44 -5.847752837517865e-14 1.0" />
         <limit/>
     </xacro:joint>
     <xacro:joint joint_name="Back_right_wheel_joint" parent_name="chassis_link" child_name="Back_right_wheel_link" joint_type="continuous" >
-        <origin xyz="-0.09000000000000004 -0.07829999999999988 0.015298850000000502" rpy="1.5707963267948317 -9.036958300754793e-32 -5.096753522204392e-16" />
-        <axis xyz="-2.0095106667766018e-44 -5.848446726908255e-14 1.0" />
+        <origin xyz="0.08999999999999966 0.07829999999999958 0.015298849999998738" rpy="-1.5707963267948446 -4.7336595440742014e-32 -3.872106723056806e-16" />
+        <axis xyz="1.5368552462246833e-44 5.848446726908255e-14 1.0" />
         <limit/>
     </xacro:joint>
     <xacro:joint joint_name="Control_left_joint" parent_name="chassis_link" child_name="Control_left_wheel_link" joint_type="revolute" >
-        <origin xyz="0.060000000000000026 0.060000000000000116 0.02579999999999962" rpy="3.141592653589787 -9.036958300754793e-32 -5.096753522204392e-16" />
-        <axis xyz="0.0 -3.469446951953671e-18 1.0" />
+        <origin xyz="-0.060000000000000386 -0.06000000000000031 0.02579999999999962" rpy="3.141592653589787 -4.7336595440742014e-32 -3.872106723056806e-16" />
+        <axis xyz="0.0 3.469446951953698e-18 1.0" />
         <limit lower="-${PI/2}" upper="${PI/2}" effort="1000000" velocity="1000000" />
     </xacro:joint>
     <xacro:joint joint_name="Front_left_wheel_joint" parent_name="Control_left_wheel_link" child_name="Front_left_wheel_link" joint_type="continuous" >
-        <origin xyz="-8.140000000009807e-06 0.005192779999999999 0.012000000000000002" rpy="3.469446951953529e-18 3.944304526105059e-31 2.0096475123297585e-44" />
-        <axis xyz="0.0 -1.0 -3.1672338534784104e-31" />
+        <origin xyz="8.140000000009807e-06 -0.005192779999999999 0.012000000000000002" rpy="-3.469446951953828e-18 7.888609052210118e-31 9.860761315264185e-32" />
+        <axis xyz="9.860761315262648e-32 1.0 1.116465887060541e-31" />
         <limit/>
     </xacro:joint>
     <xacro:joint joint_name="Control_right_joint" parent_name="chassis_link" child_name="Control_right_wheel_link" joint_type="revolute" >
-        <origin xyz="0.05999999999999998 -0.05999999999999989 0.02580000000000038" rpy="3.141592653589787 -9.036958300754793e-32 -5.096753522204392e-16" />
-        <axis xyz="0.0 -3.469446951953671e-18 1.0" />
+        <origin xyz="-0.06000000000000034 0.0599999999999997 0.025799999999998855" rpy="3.141592653589787 -4.7336595440742014e-32 -3.872106723056806e-16" />
+        <axis xyz="0.0 3.469446951953698e-18 1.0" />
         <limit lower="-${PI/2}" upper="${PI/2}" effort="1000000" velocity="1000000" />
     </xacro:joint>
     <xacro:joint joint_name="Front_right_wheel_joint" parent_name="Control_right_wheel_link" child_name="Front_right_wheel_link" joint_type="continuous" >
-        <origin xyz="-8.140000000009807e-06 0.005192779999999999 0.012000000000000002" rpy="3.469446951953529e-18 3.944304526105059e-31 2.0096475123297585e-44" />
-        <axis xyz="0.0 -1.0 -3.1672338534784104e-31" />
+        <origin xyz="8.140000000009807e-06 -0.005192779999999999 0.012000000000000002" rpy="-3.469446951953828e-18 7.888609052210118e-31 9.860761315264185e-32" />
+        <axis xyz="9.860761315262648e-32 1.0 1.116465887060541e-31" />
         <limit/>
     </xacro:joint>
     <xacro:joint joint_name="Lidar_joint" parent_name="chassis_link" child_name="Lidar_link" joint_type="fixed" >
-        <origin xyz="0.032999949999999986 -0.027999959999999404 0.09997548000000019" rpy="3.141592653589787 -9.036958300754793e-32 -5.096753522204392e-16" />
+        <origin xyz="-0.03299995000000035 0.02799996000000016 0.09997547999999906" rpy="3.141592653589787 -4.7336595440742014e-32 -3.872106723056806e-16" />
         <axis/>
         <limit/>

File: urdf/jetracer_links.xacro (robot description, xacro)
@@ -1,5 +1,5 @@
 <?xml version='1.0' encoding='utf-8'?>
 <robot xmlns:xacro="http://www.ros.org/wiki/xacro" name="jetracer">
-    <xacro:macro name="links" params="name mesh material mass *origin *inertial">
+    <xacro:macro name="links" params="name mesh material *origin *inertial">
         <link name="${name}">
             <visual name="${name}_visual">
@@ -24,73 +24,73 @@
     <!-- ================ JOINTS ================ -->
     <!-- chassis link -->
-    <xacro:links name="chassis_link" mesh="${chassis_link_mesh}" material="${chassis_link_material}" mass="${chassis_link_mass}">
+    <xacro:links name="chassis_link" mesh="${chassis_link_mesh}" material="${chassis_link_material}">
         <origin xyz="0.0 0.0 0.0" rpy="0.0 0.0 0.0" />
         <inertial>
-            <origin xyz="0.003391842842901498 -0.0016533027608844348 0.03234130593918586" rpy="0.0 0.0 0.0" />
-            <mass value="1.1769135204496393" />
-            <inertia ixx="0.0017260217976737531" iyy="0.004714734823865151" izz="0.0049585838294225635" ixy="-2.263671527874525e-05" iyz="6.326913363584177e-05" ixz="0.0003403355352982155" />
+            <origin xyz="-0.003391843429338621 0.001653302351915927 0.0323413056916162" rpy="0.0 0.0 0.0" />
+            <mass value="1.1769135087990688" />
+            <inertia ixx="0.0017260217686150478" iyy="0.004714734759311886" izz="0.004958583751749027" ixy="-2.2636682544358335e-05" iyz="-6.326912244242724e-05" ixz="-0.0003403355212436364" />
         </inertial>
     </xacro:links>
     <!-- Rear left wheel link -->
-    <xacro:links name="Back_left_wheel_link" mesh="${Back_left_wheel_mesh}" material="${Back_left_wheel_material}" mass="${Back_left_wheel_mass}">
-        <origin xyz="-3.375077994860476e-16 -8.368559845095547e-11 -3.019806626980426e-16" rpy="-3.141592653589788 -2.2183649806874918e-15 -2.1736792697780755e-29" />
+    <xacro:links name="Back_left_wheel_link" mesh="${Back_left_wheel_mesh}" material="${Back_left_wheel_material}">
+        <origin xyz="7.815970093361102e-16 8.368585602269719e-11 1.2434497875801754e-16" rpy="-3.141592653589788 2.058728436744956e-15 -1.66705181667824e-29" />
         <inertial>
-            <origin xyz="2.9305633464797864e-05 0.0004285824824775064 -0.002222785078415628" rpy="0.0 -0.0 0.0" />
+            <origin xyz="2.93056334659525e-05 0.0004285826498489609 -0.0022227850784151838" rpy="0.0 -0.0 0.0" />
             <mass value="0.054301755990382804" />
-            <inertia ixx="1.8750879631247773e-05" iyy="1.8777013070598843e-05" izz="3.0157352809619304e-05" ixy="2.018574668879972e-09" iyz="2.5074262712355275e-08" ixz="1.7150871619786058e-09" />
+            <inertia ixx="1.8750879631248003e-05" iyy="1.8777013070598626e-05" izz="3.01573528096186e-05" ixy="2.018574668852667e-09" iyz="2.507426271235245e-08" ixz="1.7150871620216485e-09" />
         </inertial>
     </xacro:links>
     <!-- Rear right wheel link -->
-    <xacro:links name="Back_right_wheel_link" mesh="${Back_right_wheel_link}" material="${Back_right_wheel_material}" mass="${Back_right_wheel_mass}">
-        <origin xyz="-3.375077994860476e-16 -8.368659543123158e-11 2.1316282072803005e-16" rpy="-5.397793497891479e-15 -2.2780382690294677e-15 3.141592653589793" />
+    <xacro:links name="Back_right_wheel_link" mesh="${Back_right_wheel_link}" material="${Back_right_wheel_material}">
+        <origin xyz="7.815970093361102e-16 8.368485904242107e-11 6.394884621840901e-16" rpy="-5.390854603987736e-15 2.4376748130006383e-15 3.141592653589793" />
         <inertial>
-            <origin xyz="-2.930563346547288e-05 0.0004285824824764406 0.0022227850784155034" rpy="0.0 -0.0 0.0" />
+            <origin xyz="-2.9305633464389303e-05 0.0004285826498478995 0.002222785078415939" rpy="0.0 -0.0 0.0" />
             <mass value="0.05430175599038278" />
-            <inertia ixx="1.8750879631247936e-05" iyy="1.877701307059906e-05" izz="3.0157352809619033e-05" ixy="-2.018574668947735e-09" iyz="-2.5074262712517995e-08" ixz="1.7150871620087073e-09" />
+            <inertia ixx="1.8750879631248153e-05" iyy="1.8777013070599494e-05" izz="3.01573528096199e-05" ixy="-2.0185746688797715e-09" iyz="-2.507426271251499e-08" ixz="1.7150871612326057e-09" />
         </inertial>
     </xacro:links>
     <!-- Front left control link -->
-    <xacro:links name="Control_left_wheel_link" mesh="${Control_left_wheel_link}" material="${Control_left_wheel_material}" mass="${Control_left_wheel_mass}">
-        <origin xyz="-8.136428598293222e-06 -0.013692779328306655 0.011999999999999334" rpy="1.570796326794897 1.5707963267948903 0" />
+    <xacro:links name="Control_left_wheel_link" mesh="${Control_left_wheel_link}" material="${Control_left_wheel_material}" >
+        <origin xyz="8.136428598790601e-06 0.013692779328306344 0.011999999999999508" rpy="-1.5707963267948961 1.5707963267948903 0" />
         <inertial>
-            <origin xyz="0.005314784577471352 -0.003309563250368317 0.012000000272431918" rpy="0.0 -0.0 0.0" />
+            <origin xyz="-0.0053147845774708545 0.003309563250368006 0.012000000272431954" rpy="0.0 -0.0 0.0" />
             <mass value="0.0022633439186205456" />
-            <inertia ixx="1.1982252143935764e-07" iyy="2.3321617796315213e-07" izz="2.609982653239135e-07" ixy="-7.588558546818486e-08" iyz="-6.531687219143192e-16" ixz="5.316366320884021e-15" />
+            <inertia ixx="1.1982252143935764e-07" iyy="2.3321617796315637e-07" izz="2.609982653239169e-07" ixy="-7.588558546818571e-08" iyz="6.531685101560824e-16" ixz="-5.316367591433442e-15" />
         </inertial>
     </xacro:links>
     <!-- Front left wheel link -->
-    <xacro:links name="Front_left_wheel_link" mesh="${Front_left_wheel_mesh}" material="${Front_left_wheel_material}" mass="${Front_left_wheel_mass}">
-        <origin xyz="3.571401290258791e-09 -0.013106999328306461 -4.019007349143067e-16" rpy="1.570796326794896 1.5707963267948843 0" />
+    <xacro:links name="Front_left_wheel_link" mesh="${Front_left_wheel_mesh}" material="${Front_left_wheel_material}">
+        <origin xyz="-3.571400783997092e-09 0.013106999328306142 -1.9761969838327787e-16" rpy="-1.5707963267948972 1.570796326794895 0" />
         <inertial>
-            <origin xyz="-0.0004285789947618479 -0.015329784406721796 -2.930563346551729e-05" rpy="0.0 -0.0 1.4597325655620378e-62" />
+            <origin xyz="0.0004285789947623453 0.015329784406721485 -2.9305633465288584e-05" rpy="0.0 -0.0 -3.335510229539365e-62" />
             <mass value="0.05430175599038286" />
-            <inertia ixx="1.8777013070599114e-05" iyy="3.0157352809619142e-05" izz="1.8750879631248044e-05" ixy="-2.5074262712421625e-08" iyz="-1.71508716181602e-09" ixz="2.0185746688459907e-09" />
+            <inertia ixx="1.877701307059917e-05" iyy="3.0157352809619196e-05" izz="1.8750879631248153e-05" ixy="-2.5074262712367415e-08" iyz="1.7150871619684858e-09" ixz="-2.018574668852767e-09" />
         </inertial>
     </xacro:links>
     <!-- Front right control link -->
-    <xacro:links name="Control_right_wheel_link" mesh="${Control_right_wheel_link}" material="${Control_right_wheel_material}" mass="${Control_right_wheel_mass}">
-        <origin xyz="-8.136428598666257e-06 0.013692779328305269 0.012000000000000144" rpy="-1.5707963267948972 -1.570796326794894 0" />
+    <xacro:links name="Control_right_wheel_link" mesh="${Control_right_wheel_link}" material="${Control_right_wheel_material}">
+        <origin xyz="8.136428599119228e-06 -0.013692779328305598 0.011999999999998564" rpy="1.5707963267948963 -1.5707963267948903 0" />
         <inertial>
-            <origin xyz="0.005314784577471317 0.0033095632503669314 0.011999999727567632" rpy="0.0 -0.0 0.0" />
+            <origin xyz="-0.005314784577470873 -0.003309563250367269 0.011999999727566086" rpy="0.0 -0.0 0.0" />
             <mass value="0.0022633439186205456" />
-            <inertia ixx="1.1982252143936103e-07" iyy="2.3321617796315552e-07" izz="2.609982653239203e-07" ixy="7.588558546818486e-08" iyz="-6.531695352472969e-16" ixz="-5.3163683852545e-15" />
+            <inertia ixx="1.1982252143937628e-07" iyy="2.3321617796315467e-07" izz="2.609982653239203e-07" ixy="7.588558546818994e-08" iyz="6.531699587637705e-16" ixz="5.316368597012737e-15" />
         </inertial>
     </xacro:links>
     <!-- Front right wheel link -->
-    <xacro:links name="Front_right_wheel_link" mesh="${Front_right_wheel_link}" material="${Front_right_wheel_material}" mass="${Front_right_wheel_mass}">
-        <origin xyz="3.5714013080223594e-09 0.01310699932830512 -3.3084646133829665e-16" rpy="-1.5707963267949037 1.5707963267948886 0" />
+    <xacro:links name="Front_right_wheel_link" mesh="${Front_right_wheel_link}" material="${Front_right_wheel_material}">
+        <origin xyz="-3.5714008195242287e-09 -0.013106999328305448 -1.942890293094024e-15" rpy="1.5707963267948892 1.5707963267948848 0" />
         <inertial>
-            <origin xyz="0.00042858613756439293 0.015329784406720446 -2.9305633465488423e-05" rpy="0.0 -0.0 0.0" />
+            <origin xyz="-0.0004285861375638955 -0.015329784406720783 -2.930563346710713e-05" rpy="0.0 -0.0 8.807362903149583e-62" />
             <mass value="0.05430175599038282" />
-            <inertia ixx="1.877701307059895e-05" iyy="3.015735280961906e-05" izz="1.8750879631247827e-05" ixy="-2.5074262712475835e-08" iyz="1.715087161843125e-09" ixz="-2.0185746688459907e-09" />
+            <inertia ixx="1.877701307059906e-05" iyy="3.0157352809619142e-05" izz="1.875087963124772e-05" ixy="-2.5074262712475835e-08" iyz="-1.7150871617821386e-09" ixz="2.018574668825662e-09" />
         </inertial>
     </xacro:links>
     <!-- Lidar link -->
-    <xacro:links name="Lidar_link" mesh="${Lidar_mesh}" material="${Lidar_material}" mass="${Lidar_mass}">
-        <origin xyz="-0.07349999799999639 -0.028000004399998054 -0.009199999999999786" rpy="3.1415926535897225 -1.936181792881828e-15 3.1415926535897927" />
+    <xacro:links name="Lidar_link" mesh="${Lidar_mesh}" material="${Lidar_material}">
+        <origin xyz="0.07349999799999678 0.028000004399998987 -0.009200000000000567" rpy="3.1415926535897354 -2.3802710027318842e-15 -3.8721067230569573e-16" />
         <inertial>
-            <origin xyz="-0.050918484442552904 -0.028239426420145132 6.461931577792513e-05" rpy="0.0 -0.0 0.0" />
+            <origin xyz="0.0509184844425533 0.0282394264201459 6.461931577717905e-05" rpy="0.0 -0.0 0.0" />
             <mass value="0.08486622487588467" />
-            <inertia ixx="2.7441257171710587e-05" iyy="7.212810687965462e-05" izz="8.077472261566907e-05" ixy="7.125364902921147e-07" iyz="-3.6800518425547077e-07" ixz="1.2837113244875235e-05" />
+            <inertia ixx="2.744125717171102e-05" iyy="7.21281068796556e-05" izz="8.077472261566873e-05" ixy="7.125364902920133e-07" iyz="3.68005184255525e-07" ixz="-1.2837113244874774e-05" />
         </inertial>
     </xacro:links>

File: urdf/jetracer_main.xacro (robot description, xacro)
@@ -25,15 +25,4 @@
     <xacro:property name="Front_right_wheel_material"   value="0.5 0.5 0.4 1" />
     <xacro:property name="Lidar_material"               value="0.5 0.5 0.4 1" />
-    <!-- ==== mass ==== -->
-    <xacro:property name="chassis_link_mass"               value="1.176913520449639" />
-    <!-- Rear -->
-    <xacro:property name="Back_left_wheel_mass"         value="0.05430175599038289" />
-    <xacro:property name="Back_right_wheel_mass"        value="0.05430175599038289" />
-    <!-- Front -->
-    <xacro:property name="Control_left_wheel_mass"      value="0.0022633439186205465" />
-    <xacro:property name="Front_left_wheel_mass"        value="0.05430175599038289" />
-    <xacro:property name="Control_right_wheel_mass"     value="0.0022633439186205465" />
-    <xacro:property name="Front_right_wheel_mass"       value="0.05430175599038289" />
-    <xacro:property name="Lidar_mass"                   value="0.08486622487588467" />
     <!-- constants -->
     <xacro:property name="PI" value="3.1415" />

Commit message: add lidar to robot and gz_bridge config file

File: urdf/jetracer_joints.xacro (robot description, xacro)
@@ -1,4 +1,4 @@
 <?xml version='1.0' encoding='utf-8'?>
-<robot xmlns:xacro="http://www.ros.org/wiki/xacro" name="jetracer">
+<robot xmlns:xacro="http://www.ros.org/wiki/xacro">
     <xacro:macro name="joint" params="joint_name parent_name child_name joint_type *origin *axis *limit">
         <xacro:property name="var" value="False"/>

File: urdf/jetracer_links.xacro (robot description, xacro)
@@ -1,4 +1,4 @@
 <?xml version='1.0' encoding='utf-8'?>
-<robot xmlns:xacro="http://www.ros.org/wiki/xacro" name="jetracer">
+<robot xmlns:xacro="http://www.ros.org/wiki/xacro">
     <xacro:macro name="links" params="name mesh material *origin *inertial">
         <link name="${name}">

File: urdf/jetracer_main.xacro (robot description, xacro)
@@ -31,4 +31,5 @@
     <xacro:include filename="jetracer_links.xacro"  />
     <xacro:include filename="jetracer_joints.xacro"  />
-    <xacro:include filename="jetracer_sensors.xacro"  />
+    <xacro:include filename="jetracer_controllers.xacro"  />
+    <xacro:include filename="jetracer_sensors.xacro" />
 </robot>

File: urdf/jetracer_sensors.xacro (robot description, xacro)
@@ -1,41 +1,26 @@
-<?xml version='1.0' encoding='utf-8'?>
-<robot xmlns:xacro="http://www.ros.org/wiki/xacro" name="jetracer">
-    <ros2_control name="GazeboSystem" type="system">
-        <hardware>
-            <plugin>gz_ros2_control/GazeboSimSystem</plugin>
-        </hardware>
-        <joint name="Back_left_wheel_joint">
-            <command_interface name="velocity" />
-            <state_interface name="velocity" />
-            <state_interface name="position" />
-        </joint>
-        <joint name="Back_right_wheel_joint">
-        <command_interface name="velocity" />
-            <state_interface name="velocity" />
-            <state_interface name="position" />
-        </joint>
-        <joint name="Control_left_joint">
-            <command_interface name="position" />
-            <state_interface name="position" />
-            <state_interface name="velocity" />
-        </joint>
-        <joint name="Control_right_joint">
-            <command_interface name="position" />
-            <state_interface name="position" />
-            <state_interface name="velocity" />
-        </joint>
-        <joint name="Front_left_wheel_joint">
-            <state_interface name="velocity"/>
-            <state_interface name="position"/>
-        </joint>
-        <joint name="Front_right_wheel_joint">
-            <state_interface name="velocity"/>
-            <state_interface name="position"/>
-        </joint>
-    </ros2_control>
-    <gazebo>
-        <plugin filename="gz_ros2_control-system" name="gz_ros2_control::GazeboSimROS2ControlPlugin">
-            <parameters>$(find jetracer_description)/config/jetracer_controller.yaml</parameters>
-        </plugin>
-  </gazebo>
+<?xml version="1.0"?>
+<robot xmlns:xacro="http://www.ros.org/wiki/xacro">
+    <gazebo reference="Lidar_link">
+        <material>Gazebo/Red</material>
+        <sensor name="laser" type="gpu_lidar">
+            <pose> 0 0 0 0 0 0 </pose>
+            <visualize>true</visualize>
+            <update_rate>10</update_rate>
+            <lidar>
+                <scan>
+                    <horizontal>
+                        <samples>360</samples>
+                        <min_angle>-3.14</min_angle>
+                        <max_angle>3.14</max_angle>
+                    </horizontal>
+                </scan>
+                <range>
+                    <min>0.3</min>
+                    <max>12</max>
+                </range>
+            </lidar>
+            <topic>scan</topic>
+            <gz_frame_id>Lidar_link</gz_frame_id>
+        </sensor>
+    </gazebo>
 </robot>
