Commit message: add camera

File: urdf/jetracer_joints.xacro (robot description, xacro)
@@ -22,35 +22,40 @@
     <!-- ================ JOINTS ================ -->
     <xacro:joint joint_name="Back_left_wheel_joint" parent_name="chassis_link" child_name="Back_left_wheel_link" joint_type="continuous" >
-        <origin xyz="0.0899999999999996 -0.07830000000000042 0.015298849999999736" rpy="-1.5707963267949614 -4.7336595440742014e-32 -3.872106723056806e-16" />
-        <axis xyz="1.5368552462246833e-44 -5.847752837517865e-14 1.0" />
+        <origin xyz="-0.09000000000000004 0.07830000000000226 0.015298849999997928" rpy="-1.570796326794903 -1.4594420859336604e-31 -3.8721067230568025e-16" />
+        <axis xyz="1.4774454646531794e-44 0.0 1.0" />
         <limit/>
     </xacro:joint>
     <xacro:joint joint_name="Back_right_wheel_joint" parent_name="chassis_link" child_name="Back_right_wheel_link" joint_type="continuous" >
-        <origin xyz="0.08999999999999966 0.07829999999999958 0.015298849999998738" rpy="-1.5707963267948446 -4.7336595440742014e-32 -3.872106723056806e-16" />
-        <axis xyz="1.5368552462246833e-44 5.848446726908255e-14 1.0" />
+        <origin xyz="-0.0900000000000001 -0.0782999999999977 0.015298849999998925" rpy="1.5707963267948317 -1.4594420859336604e-31 -3.8721067230568025e-16" />
+        <axis xyz="-1.4774454646531794e-44 -5.848446726908255e-14 1.0" />
         <limit/>
     </xacro:joint>
     <xacro:joint joint_name="Control_left_joint" parent_name="chassis_link" child_name="Control_left_wheel_link" joint_type="revolute" >
-        <origin xyz="-0.060000000000000386 -0.06000000000000031 0.02579999999999962" rpy="3.141592653589787 -4.7336595440742014e-32 -3.872106723056806e-16" />
-        <axis xyz="0.0 3.469446951953698e-18 1.0" />
+        <origin xyz="0.059999999999999956 0.060000000000002274 0.025799999999998047" rpy="3.141592653589787 -1.4594420859336604e-31 -3.8721067230568025e-16" />
+        <axis xyz="0.0 -3.469446951953726e-18 1.0" />
         <limit lower="-${PI/2}" upper="${PI/2}" effort="1000000" velocity="1000000" />
     </xacro:joint>
     <xacro:joint joint_name="Front_left_wheel_joint" parent_name="Control_left_wheel_link" child_name="Front_left_wheel_link" joint_type="continuous" >
-        <origin xyz="8.140000000009807e-06 -0.005192779999999999 0.012000000000000002" rpy="-3.469446951953828e-18 7.888609052210118e-31 9.860761315264185e-32" />
-        <axis xyz="9.860761315262648e-32 1.0 1.116465887060541e-31" />
+        <origin xyz="-8.139999999992043e-06 -0.005192779999999999 0.012000000000000002" rpy="3.46944695195376e-18 -7.888609052210118e-31 4.930380657632802e-32" />
+        <axis xyz="4.930380657631324e-32 1.0 -1.8504308629067099e-32" />
         <limit/>
     </xacro:joint>
     <xacro:joint joint_name="Control_right_joint" parent_name="chassis_link" child_name="Control_right_wheel_link" joint_type="revolute" >
-        <origin xyz="-0.06000000000000034 0.0599999999999997 0.025799999999998855" rpy="3.141592653589787 -4.7336595440742014e-32 -3.872106723056806e-16" />
-        <axis xyz="0.0 3.469446951953698e-18 1.0" />
+        <origin xyz="0.059999999999999915 -0.05999999999999773 0.02579999999999881" rpy="3.141592653589787 -1.4594420859336604e-31 -3.8721067230568025e-16" />
+        <axis xyz="0.0 -3.469446951953726e-18 1.0" />
         <limit lower="-${PI/2}" upper="${PI/2}" effort="1000000" velocity="1000000" />
     </xacro:joint>
     <xacro:joint joint_name="Front_right_wheel_joint" parent_name="Control_right_wheel_link" child_name="Front_right_wheel_link" joint_type="continuous" >
-        <origin xyz="8.140000000009807e-06 -0.005192779999999999 0.012000000000000002" rpy="-3.469446951953828e-18 7.888609052210118e-31 9.860761315264185e-32" />
-        <axis xyz="9.860761315262648e-32 1.0 1.116465887060541e-31" />
+        <origin xyz="-8.139999999992043e-06 0.005192779999999999 0.012000000000000002" rpy="3.469446951953672e-18 -7.888609052210118e-31 1.477171773546866e-44" />
+        <axis xyz="0.0 -1.0 -8.786828188924443e-32" />
         <limit/>
     </xacro:joint>
     <xacro:joint joint_name="Lidar_joint" parent_name="chassis_link" child_name="Lidar_link" joint_type="fixed" >
-        <origin xyz="-0.03299995000000035 0.02799996000000016 0.09997547999999906" rpy="3.141592653589787 -4.7336595440742014e-32 -3.872106723056806e-16" />
+        <origin xyz="0.03299994999999992 -0.027999959999997232 0.09997547999999862" rpy="3.141592653589787 -1.4594420859336604e-31 -3.8721067230568025e-16" />
+        <axis/>
+        <limit/>
+    </xacro:joint>
+    <xacro:joint joint_name="Camera_joint" parent_name="chassis_link" child_name="Camera_link" joint_type="fixed" >
+        <origin xyz="0.06897141999999992 -0.015019559999997335 0.08880616999999853" rpy="1.5707963267948903 -1.4594420859336604e-31 -3.8721067230568025e-16" />
         <axis/>
         <limit/>

File: urdf/jetracer_links.xacro (robot description, xacro)
@@ -1,19 +1,19 @@
-<?xml version='1.0' encoding='utf-8'?>
+<?xml version='1.0' encoding='utf-8' ?>
 <robot xmlns:xacro="http://www.ros.org/wiki/xacro">
     <xacro:macro name="links" params="name mesh material *origin *inertial">
         <link name="${name}">
             <visual name="${name}_visual">
-                <xacro:insert_block name="origin"/>
+                <xacro:insert_block name="origin" />
                 <geometry>
-                    <mesh filename="${mesh}" scale="${scale}"/>
+                    <mesh filename="${mesh}" scale="${scale}" />
                 </geometry>
                 <material name="${name}_material">
-                    <color rgba="${material}"/>
+                    <color rgba="${material}" />
                 </material>
             </visual>
             <collision name="${name}_collision">
-                <xacro:insert_block name="origin"/>
+                <xacro:insert_block name="origin" />
                 <geometry>
-                    <mesh filename="${mesh}" scale="${scale}"/>
+                    <mesh filename="${mesh}" scale="${scale}" />
                 </geometry>
             </collision>
@@ -24,73 +24,228 @@
     <!-- ================ JOINTS ================ -->
     <!-- chassis link -->
-    <xacro:links name="chassis_link" mesh="${chassis_link_mesh}" material="${chassis_link_material}">
+    <xacro:links
+        name="chassis_link"
+        mesh="${chassis_link_mesh}"
+        material="${chassis_link_material}"
+    >
         <origin xyz="0.0 0.0 0.0" rpy="0.0 0.0 0.0" />
         <inertial>
-            <origin xyz="-0.003391843429338621 0.001653302351915927 0.0323413056916162" rpy="0.0 0.0 0.0" />
-            <mass value="1.1769135087990688" />
-            <inertia ixx="0.0017260217686150478" iyy="0.004714734759311886" izz="0.004958583751749027" ixy="-2.2636682544358335e-05" iyz="-6.326912244242724e-05" ixz="-0.0003403355212436364" />
+            <origin xyz="0.0 0.0 0.0" rpy="0.0 0.0 0.0" />
+            <mass value="1.1691869669622004" />
+            <inertia
+                ixx="0.0016985538990736126"
+                iyy="0.004643646847817014"
+                izz="0.004914083439210598"
+                ixy="-2.1598217488998493e-05"
+                iyz="6.408477724474828e-05"
+                ixz="0.00037447818172130085"
+            />
         </inertial>
     </xacro:links>
     <!-- Rear left wheel link -->
-    <xacro:links name="Back_left_wheel_link" mesh="${Back_left_wheel_mesh}" material="${Back_left_wheel_material}">
-        <origin xyz="7.815970093361102e-16 8.368585602269719e-11 1.2434497875801754e-16" rpy="-3.141592653589788 2.058728436744956e-15 -1.66705181667824e-29" />
-        <inertial>
-            <origin xyz="2.93056334659525e-05 0.0004285826498489609 -0.0022227850784151838" rpy="0.0 -0.0 0.0" />
+    <xacro:links
+        name="Back_left_wheel_link"
+        mesh="${Back_left_wheel_mesh}"
+        material="${Back_left_wheel_material}"
+    >
+        <origin
+            xyz="-2.486899575160351e-16 8.368400861158421e-11 -1.8118839761882555e-15"
+            rpy="6.413861609175051e-14 2.9122543710783113e-15 2.116368867342585e-28"
+        />
+        <inertial>
+            <origin
+                xyz="2.930563346486892e-05 -0.000428582482479225 0.0022227850784134516"
+                rpy="0.0 -0.0 0.0"
+            />
             <mass value="0.054301755990382804" />
-            <inertia ixx="1.8750879631248003e-05" iyy="1.8777013070598626e-05" izz="3.01573528096186e-05" ixy="2.018574668852667e-09" iyz="2.507426271235245e-08" ixz="1.7150871620216485e-09" />
+            <inertia
+                ixx="1.8750879631248586e-05"
+                iyy="1.8777013070599494e-05"
+                izz="3.0157352809618708e-05"
+                ixy="-2.0185746688392145e-09"
+                iyz="2.5074262711716894e-08"
+                ixz="-1.7150871619176639e-09"
+            />
         </inertial>
     </xacro:links>
     <!-- Rear right wheel link -->
-    <xacro:links name="Back_right_wheel_link" mesh="${Back_right_wheel_link}" material="${Back_right_wheel_material}">
-        <origin xyz="7.815970093361102e-16 8.368485904242107e-11 6.394884621840901e-16" rpy="-5.390854603987736e-15 2.4376748130006383e-15 3.141592653589793" />
-        <inertial>
-            <origin xyz="-2.9305633464389303e-05 0.0004285826498478995 0.002222785078415939" rpy="0.0 -0.0 0.0" />
+    <xacro:links
+        name="Back_right_wheel_link"
+        mesh="${Back_right_wheel_link}"
+        material="${Back_right_wheel_material}"
+    >
+        <origin
+            xyz="-1.7763568394002506e-16 -8.368500337141427e-11 2.3803181647963358e-15"
+            rpy="7.311237941014883e-15 2.488315143520874e-15 3.834643568612533e-29"
+        />
+        <inertial>
+            <origin
+                xyz="2.93056334649755e-05 -0.0004285826498480705 0.0022227850784176974"
+                rpy="0.0 -0.0 0.0"
+            />
             <mass value="0.05430175599038278" />
-            <inertia ixx="1.8750879631248153e-05" iyy="1.8777013070599494e-05" izz="3.01573528096199e-05" ixy="-2.0185746688797715e-09" iyz="-2.507426271251499e-08" ixz="1.7150871612326057e-09" />
+            <inertia
+                ixx="1.875087963124772e-05"
+                iyy="1.8777013070598626e-05"
+                izz="3.0157352809619142e-05"
+                ixy="-2.0185746689610867e-09"
+                iyz="2.5074262712379465e-08"
+                ixz="-1.7150871619892508e-09"
+            />
         </inertial>
     </xacro:links>
     <!-- Front left control link -->
-    <xacro:links name="Control_left_wheel_link" mesh="${Control_left_wheel_link}" material="${Control_left_wheel_material}" >
-        <origin xyz="8.136428598790601e-06 0.013692779328306344 0.011999999999999508" rpy="-1.5707963267948961 1.5707963267948903 0" />
-        <inertial>
-            <origin xyz="-0.0053147845774708545 0.003309563250368006 0.012000000272431954" rpy="0.0 -0.0 0.0" />
+    <xacro:links
+        name="Control_left_wheel_link"
+        mesh="${Control_left_wheel_link}"
+        material="${Control_left_wheel_material}"
+    >
+        <origin
+            xyz="-8.136428598213286e-06 -0.013692779328304639 0.011999999999997783"
+            rpy="1.570796326794897 1.5707963267948903 0"
+        />
+        <inertial>
+            <origin
+                xyz="0.005314784577471432 -0.0033095632503662743 0.012000000272430367"
+                rpy="0.0 -0.0 0.0"
+            />
             <mass value="0.0022633439186205456" />
-            <inertia ixx="1.1982252143935764e-07" iyy="2.3321617796315637e-07" izz="2.609982653239169e-07" ixy="-7.588558546818571e-08" iyz="6.531685101560824e-16" ixz="-5.316367591433442e-15" />
+            <inertia
+                ixx="1.1982252143944404e-07"
+                iyy="2.3321617796315722e-07"
+                izz="2.609982653239474e-07"
+                ixy="-7.5885585468173e-08"
+                iyz="-6.531708057967177e-16"
+                ixz="5.316366267672132e-15"
+            />
         </inertial>
     </xacro:links>
     <!-- Front left wheel link -->
-    <xacro:links name="Front_left_wheel_link" mesh="${Front_left_wheel_mesh}" material="${Front_left_wheel_material}">
-        <origin xyz="-3.571400783997092e-09 0.013106999328306142 -1.9761969838327787e-16" rpy="-1.5707963267948972 1.570796326794895 0" />
-        <inertial>
-            <origin xyz="0.0004285789947623453 0.015329784406721485 -2.9305633465288584e-05" rpy="0.0 -0.0 -3.335510229539365e-62" />
+    <xacro:links
+        name="Front_left_wheel_link"
+        mesh="${Front_left_wheel_mesh}"
+        material="${Front_left_wheel_material}"
+    >
+        <origin
+            xyz="3.5714013080223594e-09 -0.013106999328304383 -2.0050627824730326e-15"
+            rpy="1.570796326794896 1.5707963267948843 0"
+        />
+        <inertial>
+            <origin
+                xyz="-0.00042857899476183013 -0.015329784406719754 -2.930563346712267e-05"
+                rpy="0.0 -0.0 1.4597325655614851e-62"
+            />
             <mass value="0.05430175599038286" />
-            <inertia ixx="1.877701307059917e-05" iyy="3.0157352809619196e-05" izz="1.8750879631248153e-05" ixy="-2.5074262712367415e-08" iyz="1.7150871619684858e-09" ixz="-2.018574668852767e-09" />
+            <inertia
+                ixx="1.877701307059689e-05"
+                iyy="3.0157352809619223e-05"
+                izz="1.8750879631245117e-05"
+                ixy="-2.5074262712584255e-08"
+                iyz="-1.7150871617550335e-09"
+                ixz="2.0185746688392145e-09"
+            />
         </inertial>
     </xacro:links>
     <!-- Front right control link -->
-    <xacro:links name="Control_right_wheel_link" mesh="${Control_right_wheel_link}" material="${Control_right_wheel_material}">
-        <origin xyz="8.136428599119228e-06 -0.013692779328305598 0.011999999999998564" rpy="1.5707963267948963 -1.5707963267948903 0" />
-        <inertial>
-            <origin xyz="-0.005314784577470873 -0.003309563250367269 0.011999999727566086" rpy="0.0 -0.0 0.0" />
+    <xacro:links
+        name="Control_right_wheel_link"
+        mesh="${Control_right_wheel_link}"
+        material="${Control_right_wheel_material}"
+    >
+        <origin
+            xyz="-8.136428598497503e-06 0.013692779328307196 0.011999999999998732"
+            rpy="-1.570796326794897 -1.5707963267948903 0"
+        />
+        <inertial>
+            <origin
+                xyz="0.005314784577471485 0.0033095632503688677 0.011999999727566124"
+                rpy="0.0 -0.0 0.0"
+            />
             <mass value="0.0022633439186205456" />
-            <inertia ixx="1.1982252143937628e-07" iyy="2.3321617796315467e-07" izz="2.609982653239203e-07" ixy="7.588558546818994e-08" iyz="6.531699587637705e-16" ixz="5.316368597012737e-15" />
+            <inertia
+                ixx="1.1982252143934917e-07"
+                iyy="2.3321617796315552e-07"
+                izz="2.6099826532390675e-07"
+                ixy="7.588558546818994e-08"
+                iyz="-6.531691454307929e-16"
+                ixz="-5.316368438466389e-15"
+            />
         </inertial>
     </xacro:links>
     <!-- Front right wheel link -->
-    <xacro:links name="Front_right_wheel_link" mesh="${Front_right_wheel_link}" material="${Front_right_wheel_material}">
-        <origin xyz="-3.5714008195242287e-09 -0.013106999328305448 -1.942890293094024e-15" rpy="1.5707963267948892 1.5707963267948848 0" />
-        <inertial>
-            <origin xyz="-0.0004285861375638955 -0.015329784406720783 -2.930563346710713e-05" rpy="0.0 -0.0 8.807362903149583e-62" />
+    <xacro:links
+        name="Front_right_wheel_link"
+        mesh="${Front_right_wheel_link}"
+        material="${Front_right_wheel_material}"
+    >
+        <origin
+            xyz="3.5714013879584174e-09 0.013106999328307153 -1.7341683644644946e-15"
+            rpy="-1.5707963267949039 1.5707963267948957 0"
+        />
+        <inertial>
+            <origin
+                xyz="0.00042858613756447284 0.015329784406722453 -2.930563346686954e-05"
+                rpy="0.0 -0.0 0.0"
+            />
             <mass value="0.05430175599038282" />
-            <inertia ixx="1.877701307059906e-05" iyy="3.0157352809619142e-05" izz="1.875087963124772e-05" ixy="-2.5074262712475835e-08" iyz="-1.7150871617821386e-09" ixz="2.018574668825662e-09" />
+            <inertia
+                ixx="1.8777013070598843e-05"
+                iyy="3.0157352809619142e-05"
+                izz="1.8750879631247936e-05"
+                ixy="-2.5074262712584255e-08"
+                iyz="1.715087161971874e-09"
+                ixz="-2.0185746688459907e-09"
+            />
         </inertial>
     </xacro:links>
     <!-- Lidar link -->
-    <xacro:links name="Lidar_link" mesh="${Lidar_mesh}" material="${Lidar_material}">
-        <origin xyz="0.07349999799999678 0.028000004399998987 -0.009200000000000567" rpy="3.1415926535897354 -2.3802710027318842e-15 -3.8721067230569573e-16" />
-        <inertial>
-            <origin xyz="0.0509184844425533 0.0282394264201459 6.461931577717905e-05" rpy="0.0 -0.0 0.0" />
+    <xacro:links
+        name="Lidar_link"
+        mesh="${Lidar_mesh}"
+        material="${Lidar_material}"
+    >
+        <origin
+            xyz="-0.07349999799999625 -0.028000004399996004 -0.009200000000001455"
+            rpy="3.1415926535897225 -1.9361817928818287e-15 3.1415926535897927"
+        />
+        <inertial>
+            <origin
+                xyz="-0.050918484442552744 -0.028239426420143127 6.461931577627312e-05"
+                rpy="0.0 -0.0 0.0"
+            />
             <mass value="0.08486622487588467" />
-            <inertia ixx="2.744125717171102e-05" iyy="7.21281068796556e-05" izz="8.077472261566873e-05" ixy="7.125364902920133e-07" iyz="3.68005184255525e-07" ixz="-1.2837113244874774e-05" />
+            <inertia
+                ixx="2.7441257171710587e-05"
+                iyy="7.212810687965495e-05"
+                izz="8.07747226156683e-05"
+                ixy="7.125364902921759e-07"
+                iyz="-3.680051842555253e-07"
+                ixz="1.2837113244875167e-05"
+            />
+        </inertial>
+    </xacro:links>
+    <xacro:links
+        name="Camera_link"
+        mesh="${Camera_mesh}"
+        material="${Camera_material}"
+    >
+        <origin
+            xyz="0.0049999959182071676 -0.00319999685272796 -0.014299990434673546"
+            rpy="-1.5707963267948897 6.455673410932649e-14 4.110951392333017e-28"
+        />
+        <inertial>
+            <origin
+                xyz="0.009437076326469703 -0.00214409346072566 -0.014385412303800145"
+                rpy="0.0 -0.0 0.0"
+            />
+            <mass value="0.007726553487439356" />
+            <inertia
+                ixx="7.268716244665518e-07"
+                iyy="7.070297059504462e-07"
+                izz="6.032871415961253e-07"
+                ixy="-5.27821034369442e-08"
+                iyz="8.56540756914324e-10"
+                ixz="4.390662029237586e-09"
+            />
         </inertial>
     </xacro:links>
