Commit message: add camera

File: urdf/jetracer_main.xacro (robot description, xacro)
@@ -1,35 +1,55 @@
-<?xml version='1.0' encoding='utf-8'?>
+<?xml version='1.0' encoding='utf-8' ?>
 <robot xmlns:xacro="http://www.ros.org/wiki/xacro" name="jetracer">
     <!-- ================= PROPERTIES ================== -->
     <xacro:property name="scale" value="0.001 0.001 0.001" />
     <!-- ==== meshes ==== -->
-    <xacro:property name="chassis_link_mesh"               value="file://$(find jetracer_description)/meshes/Base_link.stl" />
+    <xacro:property
+        name="chassis_link_mesh"
+        value="file://$(find jetracer_description)/meshes/Base_link.stl"/>
     <!-- Rear -->
-    <xacro:property name="Back_left_wheel_mesh"         value="file://$(find jetracer_description)/meshes/Back_left_wheel_link.stl" />
-    <xacro:property name="Back_right_wheel_link"        value="file://$(find jetracer_description)/meshes/Back_right_wheel_link.stl" />
+    <xacro:property
+        name="Back_left_wheel_mesh"
+        value="file://$(find jetracer_description)/meshes/Back_left_wheel_link.stl"/>
+    <xacro:property
+        name="Back_right_wheel_link"
+        value="file://$(find jetracer_description)/meshes/Back_right_wheel_link.stl"/>
     <!-- Front -->
-    <xacro:property name="Control_left_wheel_link"      value="file://$(find jetracer_description)/meshes/Control_right_wheel_link.stl" />
-    <xacro:property name="Front_left_wheel_mesh"        value="file://$(find jetracer_description)/meshes/Front_left_wheel_link.stl" />
-    <xacro:property name="Control_right_wheel_link"     value="file://$(find jetracer_description)/meshes/Control_right_wheel_link.stl" />
-    <xacro:property name="Front_right_wheel_link"       value="file://$(find jetracer_description)/meshes/Front_right_wheel_link.stl" />
-    <xacro:property name="Lidar_mesh"                   value="file://$(find jetracer_description)/meshes/Lidar_link.stl" />
+    <xacro:property
+        name="Control_left_wheel_link"
+        value="file://$(find jetracer_description)/meshes/Control_right_wheel_link.stl"/>
+    <xacro:property
+        name="Front_left_wheel_mesh"
+        value="file://$(find jetracer_description)/meshes/Front_left_wheel_link.stl"/>
+    <xacro:property
+        name="Control_right_wheel_link"
+        value="file://$(find jetracer_description)/meshes/Control_right_wheel_link.stl"/>
+    <xacro:property
+        name="Front_right_wheel_link"
+        value="file://$(find jetracer_description)/meshes/Front_right_wheel_link.stl"/>
+    <xacro:property
+        name="Lidar_mesh"
+        value="file://$(find jetracer_description)/meshes/Lidar_link.stl"/>
+    <xacro:property
+        name="Camera_mesh"
+        value="file://$(find jetracer_description)/meshes/Camera.stl"/>
     <!-- ==== materials ==== -->
-    <xacro:property name="chassis_link_material"           value="0.25 0.25 0.25 1" />
+    <xacro:property name="chassis_link_material" value="0.25 0.25 0.25 1" />
     <!-- Rear -->
-    <xacro:property name="Back_left_wheel_material"     value="0.5 0.5 0.4 1" />
-    <xacro:property name="Back_right_wheel_material"    value="0.5 0.5 0.4 1" />
+    <xacro:property name="Back_left_wheel_material" value="0.5 0.5 0.4 1" />
+    <xacro:property name="Back_right_wheel_material" value="0.5 0.5 0.4 1" />
     <!-- Front -->
-    <xacro:property name="Control_left_wheel_material"  value="0.5 0.5 0.4 1" />
-    <xacro:property name="Front_left_wheel_material"    value="0.5 0.5 0.4 1" />
+    <xacro:property name="Control_left_wheel_material" value="0.5 0.5 0.4 1" />
+    <xacro:property name="Front_left_wheel_material" value="0.5 0.5 0.4 1" />
     <xacro:property name="Control_right_wheel_material" value="0.5 0.5 0.4 1" />
-    <xacro:property name="Front_right_wheel_material"   value="0.5 0.5 0.4 1" />
-    <xacro:property name="Lidar_material"               value="0.5 0.5 0.4 1" />
+    <xacro:property name="Front_right_wheel_material" value="0.5 0.5 0.4 1" />
+    <xacro:property name="Lidar_material" value="0.5 0.5 0.4 1" />
+    <xacro:property name="Camera_material" value="0.5 0.5 0.4 1" />
     <!-- constants -->
     <xacro:property name="PI" value="3.1415" />
     <xacro:property name="scale" value="0.001 0.001 0.001" />
     <!-- ================= INCLUDES ================== -->
-    <xacro:include filename="jetracer_links.xacro"  />
-    <xacro:include filename="jetracer_joints.xacro"  />
-    <xacro:include filename="jetracer_controllers.xacro"  />
+    <xacro:include filename="jetracer_links.xacro" />
+    <xacro:include filename="jetracer_joints.xacro" />
+    <xacro:include filename="jetracer_controllers.xacro" />
     <xacro:include filename="jetracer_sensors.xacro" />
 </robot>

File: urdf/jetracer_sensors.xacro (robot description, xacro)
@@ -24,3 +24,38 @@
         </sensor>
     </gazebo>
+    <joint name="camera_joint" type="fixed">
+        <parent link="Camera_link"/>
+        <child link="camera_link"/>
+        <origin xyz="0.015019559999997335 0.00105 -0.015019555" rpy="-1.5707963267948903 1.4594420859336604e-31 3.8721067230568025e-16"/>
+    </joint>
+    <link name="camera_link"/>
+    <joint name="camera_optical_joint" type="fixed">
+        <parent link="camera_link"/>
+        <child link="camera_link_optical"/>
+        <origin xyz="0 0 0" rpy="${-pi/2} 0 ${-pi/2}"/>
+    </joint>
+    <link name="camera_link_optical"/>
+    <gazebo reference="camera_link">
+        <material>Gazebo/Red</material>
+        <sensor name="camera" type="camera">
+            <pose> 0 0 0 0 0 0 </pose>
+            <visualize>true</visualize>
+            <update_rate>10</update_rate>
+            <camera>
+                <camera_info_topic>camera/camera_info</camera_info_topic>
+                <horizontal_fov>1.089</horizontal_fov>
+                <image>
+                    <format>R8G8B8</format>
+                    <width>640</width>
+                    <height>480</height>
+                </image>
+                <clip>
+                    <near>0.05</near>
+                    <far>8.0</far>
+                </clip>
+            </camera>
+            <topic>camera/image_raw</topic>
+            <gz_frame_id>camera_link_optical</gz_frame_id>
+        </sensor>
+    </gazebo>
 </robot>

Commit message: fix rear wheel direction

File: urdf/jetracer_joints.xacro (robot description, xacro)
@@ -28,5 +28,5 @@
     <xacro:joint joint_name="Back_right_wheel_joint" parent_name="chassis_link" child_name="Back_right_wheel_link" joint_type="continuous" >
         <origin xyz="-0.0900000000000001 -0.0782999999999977 0.015298849999998925" rpy="1.5707963267948317 -1.4594420859336604e-31 -3.8721067230568025e-16" />
-        <axis xyz="-1.4774454646531794e-44 -5.848446726908255e-14 1.0" />
+        <axis xyz="-1.4774454646531794e-44 -5.848446726908255e-14 -1.0" />
         <limit/>
     </xacro:joint>
