Commit message: add joystick scripts

File: jetracer_description/urdf/jetracer_joints.xacro (robot description, xacro)
@@ -16,8 +16,18 @@
     </xacro:macro>
     <joint name="chassis_joint" type="fixed">
-    <origin xyz="0 0 0" rpy="0 0 0" />
-    <parent link="base_link" />
-    <child link="chassis_link" />
-  </joint>
+        <origin xyz="0 0 0" rpy="0 0 0" />
+        <parent link="base_link" />
+        <child link="chassis_link" />
+    </joint>
+    <joint name="base_footprint_joint" type="fixed">
+        <origin xyz="0 0 0" rpy="0 0 0" />
+        <parent link="base_link" />
+        <child link="base_footprint" />
+    </joint>
+    <joint name="laser_joint" type="fixed">
+        <origin xyz="0.005 0 0.120" rpy="0 0 0" />
+        <parent link="base_link" />
+        <child link="laser" />
+    </joint>
     <!-- ================ JOINTS ================ -->
     <xacro:joint joint_name="Back_left_wheel_joint" parent_name="chassis_link" child_name="Back_left_wheel_link" joint_type="continuous" >

File: jetracer_description/urdf/jetracer_links.xacro (robot description, xacro)
@@ -22,4 +22,6 @@
     </xacro:macro>
     <link name="base_link" />
+    <link name="base_footprint" />
+    <link name="laser" />
     <!-- ================ JOINTS ================ -->
     <!-- chassis link -->

Commit message: fix urdf axes

File: jetracer_description/urdf/jetracer_joints.xacro (robot description, xacro)
@@ -43,6 +43,6 @@
     <xacro:joint joint_name="Control_left_joint" parent_name="chassis_link" child_name="Control_left_wheel_link" joint_type="revolute" >
         <origin xyz="0.059999999999999956 0.060000000000002274 0.025799999999998047" rpy="3.141592653589787 -1.4594420859336604e-31 -3.8721067230568025e-16" />
-        <axis xyz="0.0 -3.469446951953726e-18 1.0" />
-        <limit lower="-${PI/2}" upper="${PI/2}" effort="1000000" velocity="1000000" />
+        <axis xyz="0.0 0.0 -1.0" />
+        <limit lower="-${PI/4}" upper="${PI/4}" effort="1000000" velocity="1000000" />
     </xacro:joint>
     <xacro:joint joint_name="Front_left_wheel_joint" parent_name="Control_left_wheel_link" child_name="Front_left_wheel_link" joint_type="continuous" >
@@ -53,6 +53,6 @@
     <xacro:joint joint_name="Control_right_joint" parent_name="chassis_link" child_name="Control_right_wheel_link" joint_type="revolute" >
         <origin xyz="0.059999999999999915 -0.05999999999999773 0.02579999999999881" rpy="3.141592653589787 -1.4594420859336604e-31 -3.8721067230568025e-16" />
-        <axis xyz="0.0 -3.469446951953726e-18 1.0" />
-        <limit lower="-${PI/2}" upper="${PI/2}" effort="1000000" velocity="1000000" />
+        <axis xyz="0.0 0.0 -1.0" />
+        <limit lower="-${PI/4}" upper="${PI/4}" effort="1000000" velocity="1000000" />
     </xacro:joint>
     <xacro:joint joint_name="Front_right_wheel_joint" parent_name="Control_right_wheel_link" child_name="Front_right_wheel_link" joint_type="continuous" >

File: jetracer_description/urdf/jetracer_sensors.xacro (robot description, xacro)
@@ -1,5 +1,5 @@
 <?xml version="1.0"?>
 <robot xmlns:xacro="http://www.ros.org/wiki/xacro">
-    <gazebo reference="Lidar_link">
+    <gazebo reference="laser">
         <material>Gazebo/Red</material>
         <sensor name="laser" type="gpu_lidar">
@@ -21,5 +21,5 @@
             </lidar>
             <topic>scan</topic>
-            <gz_frame_id>Lidar_link</gz_frame_id>
+            <gz_frame_id>laser</gz_frame_id>
         </sensor>
     </gazebo>

Commit message: streamlining mapper for hardware and sim

File: jetracer_description/urdf/jetracer_joints.xacro (robot description, xacro)
@@ -25,8 +25,27 @@
         <child link="base_footprint" />
     </joint>
-    <joint name="laser_joint" type="fixed">
-        <origin xyz="0.005 0 0.120" rpy="0 0 0" />
-        <parent link="base_link" />
-        <child link="laser" />
+    <xacro:if value="$(arg use_sim)">
+        <joint name="laser_joint" type="fixed">
+            <origin xyz="0.005 0 0.120" rpy="0 0 0" />
+            <parent link="base_link" />
+            <child link="laser" />
+        </joint>
+    </xacro:if>
+    <xacro:unless value="$(arg use_sim)">
+        <joint name="laser_joint" type="fixed">
+            <origin xyz="0.005 0 0.120" rpy="0 0 ${pi}" />
+            <parent link="base_link" />
+            <child link="laser" />
+        </joint>
+    </xacro:unless>
+    <joint name="camera_joint" type="fixed">
+        <parent link="Camera_link"/>
+        <child link="camera_link"/>
+        <origin xyz="0.015019559999997335 0.00105 -0.015019555" rpy="-1.5707963267948903 1.4594420859336604e-31 3.8721067230568025e-16"/>
+    </joint>
+    <joint name="camera_optical_joint" type="fixed">
+        <parent link="camera_link"/>
+        <child link="camera_link_optical"/>
+        <origin xyz="0 0 0" rpy="${-pi/2} 0 ${-pi/2}"/>
     </joint>
     <!-- ================ JOINTS ================ -->

File: jetracer_description/urdf/jetracer_links.xacro (robot description, xacro)
@@ -33,4 +33,6 @@
     <link name="base_footprint" />
     <link name="laser" />
+    <link name="camera_link"/>
+    <link name="camera_link_optical"/>
     <!-- ================ JOINTS ================ -->
     <!-- chassis link -->

File: jetracer_description/urdf/jetracer_main.xacro (robot description, xacro)
@@ -3,4 +3,5 @@
     <!-- ================= ARGUMENTS  ================== -->
     <xacro:arg name="namespace" default="jetracer" />
+    <xacro:arg name="use_sim" default="true"/>
     <!-- ================= PROPERTIES ================== -->
     <xacro:property name="scale" value="0.001 0.001 0.001" />
@@ -53,5 +54,7 @@
     <xacro:include filename="jetracer_links.xacro" />
     <xacro:include filename="jetracer_joints.xacro" />
-    <xacro:include filename="jetracer_controllers.xacro" />
-    <xacro:include filename="jetracer_sensors.xacro" />
+    <xacro:if value="$(arg use_sim)">
+        <xacro:include filename="jetracer_controllers.xacro" />
+        <xacro:include filename="jetracer_sensors.xacro" />
+    </xacro:if>
 </robot>

File: jetracer_description/urdf/jetracer_sensors.xacro (robot description, xacro)
@@ -24,16 +24,4 @@
         </sensor>
     </gazebo>
-    <joint name="camera_joint" type="fixed">
-        <parent link="Camera_link"/>
-        <child link="camera_link"/>
-        <origin xyz="0.015019559999997335 0.00105 -0.015019555" rpy="-1.5707963267948903 1.4594420859336604e-31 3.8721067230568025e-16"/>
-    </joint>
-    <link name="camera_link"/>
-    <joint name="camera_optical_joint" type="fixed">
-        <parent link="camera_link"/>
-        <child link="camera_link_optical"/>
-        <origin xyz="0 0 0" rpy="${-pi/2} 0 ${-pi/2}"/>
-    </joint>
-    <link name="camera_link_optical"/>
     <gazebo reference="camera_link">
         <material>Gazebo/Red</material>
